File: PCB Shield/Mega_2560_core_mini_full_2.0_B/Mega_2560 core mini_full_2.0-B.kicad_pcb (KiCad board)
At the start: 2 copper layers, 99 parts, among them P1 2560-core, P10 SPI_libre, P11 Trim, P12 Stick_left, P13 Stick_right, P14 Switch, P15 LCD_I2C, P16 LCD, P17 Battery LIPO, P18 Ecolage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

Commit message: Update_Mega_2560_core_mini_full_2.0-B
Parts:
- added C10: 47µF, Capacitors_SMD:CP_Elec_6.3x5.3, B.Cu at (221.6, 71.4)
- added C2: 47nF, Capacitors_SMD:C_1206, F.Cu at (122.3, 73.9)
- added C7: 100nF, Capacitors_SMD:C_1206, F.Cu at (126.7, 114.6)
- added C8: 47µF, Capacitors_SMD:CP_Elec_6.3x5.3, B.Cu at (223.0, 83.5)
- added P3: Option, Pin_Headers:Pin_Header_Straight_1x04_Pitch2.54mm, F.Cu at (154.9, 115.2)
- added P7: Option, Pin_Headers:Pin_Header_Straight_1x06_Pitch2.54mm, F.Cu at (179.7, 77.1)
- C43, C44, C45, C46: value 22nF -> 4.7nF
- R11, R12, R13, R14: value 15K -> 100K
- R26, R29, R32, R35: value 10K -> 47K
- R27, R30, R33, R36: value POT_22k -> POT_100k
- R28, R31, R34, R37: value 10K -> 270K
- R7: value 500 -> 470
- RV1: footprint Potentiometers:Potentiometer_Triwood_RM-065 -> Potentiometers:Potentiometer_Trimmer_Bourns_3214W
- RV2, RV3, RV4, RV5: footprint Potentiometers:Potentiometer_Bourns_3296W_3-8Zoll_Inline_ScrewUp -> Potentiometers:Potentiometer_Trimmer_Bourns_3296W
- RV6: footprint Potentiometers:Potentiometer_Trimmer_Bourns_3266W -> Potentiometers:Potentiometer_Trimmer_Bourns_3214W
- U2, U3: footprint anthoperso:SOP4 -> Librairie master:SOP4
- moved RV6 68.3 mm to (131.4, 100.6)
- moved C4 42.6 mm to (113.6, 105.1)
- moved RV1 26.5 mm to (130.1, 87.2)
- moved C6 19.6 mm to (121.3, 90.5)
- moved P2 0.64 mm to (154.9, 119.0)
- moved U2 0.63 mm to (214.0, 98.1), turned to 90 degrees
- turned RV2 to 0 degrees
- turned RV3 to 0 degrees
- turned RV4 to 0 degrees
- turned RV5 to 0 degrees
- turned U3 to 90 degrees
Connections:
- C45 pad 1: /Stick_LV -> /Stick_LH
- C46 pad 1: /Stick_LH -> /Stick_LV
- P20 pad 4: /RX_module -> Net-(P20-Pad4)
- P20 pad 5: Net-(P20-Pad5) -> GND
- P20 pad 6: /TX_module -> VCC
- P20 pad 7: VCC -> /TX_module
- P20 pad 8: GND -> /RX_module
- R32 pad 2: /Stick_LVcon -> /Stick_LHcon
- R33 pad 2: /Stick_LV -> /Stick_LH
- R33 pad 3: /Stick_LV -> /Stick_LH
- R35 pad 2: /Stick_LHcon -> /Stick_LVcon
- R36 pad 2: /Stick_LH -> /Stick_LV
- R36 pad 3: /Stick_LH -> /Stick_LV
- U3 pad 4: Net-(P20-Pad5) -> Net-(P20-Pad4)
- U6 pad 14: /Stick_LH -> /Stick_LV
- U6 pad 8: /Stick_LV -> /Stick_LH
- W3 pad 1: /Stick_LV -> /Stick_LH
- W3 pad 2: /Stick_LVcon -> /Stick_LHcon
- W4 pad 1: /Stick_LH -> /Stick_LV
- W4 pad 2: /Stick_LHcon -> /Stick_LVcon
Routing:
- net VCC: track 321.1 -> 377.0 mm, vias 2 -> 4
- net /audio_right_in: track 38.9 -> 0.00 mm, vias 1 -> 0
- net /PPM_TX_OUT: track 0.00 -> 35.2 mm, vias 0 -> 3
- net /Microsd_CS: track 0.00 -> 33.9 mm, vias 0 -> 1
- net /PPM_out: track 0.00 -> 28.5 mm, vias 0 -> 4
- net /Stick_LV: track 51.2 -> 28.7 mm, vias 4 -> 1
- net Net-(P22-PadRX): track 32.9 -> 13.7 mm
- net /PPM_in: track 0.00 -> 14.6 mm
- net Net-(P20-Pad5): track 13.9 -> 0.00 mm
- net /Sim_control: track 0.00 -> 13.7 mm, vias 0 -> 2
- net /Stick_LVcon: track 23.7 -> 10.2 mm, vias 2 -> 1
- net /Lcd_bla: track 13.3 -> 0.00 mm, vias 1 -> 0
- net GND: track 77.7 -> 90.3 mm, vias 8 -> 10
- net Net-(D1-Pad1): track 0.00 -> 12.1 mm, vias 0 -> 1
- net /Stick_LH: track 41.3 -> 29.2 mm, vias 3 -> 2
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