File: PCB Shield/Mega_2560_core_mini_full_2.0_B/Mega_2560 core mini_full_2.0-B.sch (KiCad schematic (older format))
At the start: 105 parts, among them P1 2560-core, P10 SPI_libre, P11 Trim, P12 Stick_left, P13 Stick_right, P14 Switch, P15 LCD_I2C, P16 LCD, P17 Battery LIPO, P18 Ecolage, P19 Module_TX, P2 Clock, P20 Module_RS232/TTL, P21 Sw_power, P22 CONN_JQ6500_28P_mini, P23 Rot_1, P24 Rot_2, P25 Key_select_menu_ESC, P26 LCD_Vcc_select, P3 Option, P4 Potentiometre, P5 Vibreur, P6 Micro_sd, P7 Option, P8 Audio, P9 SPI, SW1 Inter_HF, SW3 Power switch, U1 4066, U2 TLP290, U3 TLP290, U4 L4941, U5 LD1117S33TR, U6 MCP604-I/SL

Commit message: Update_Mega_2560_core_mini_full_2.0-B
Parts:
- removed SW1: Inter_HF, symbol SW_DPST_x2
- removed SW3: Power switch, symbol SW_DPST_x2
- added C10, C8: 47µF, Capacitors_SMD:CP_Elec_6.3x5.3, symbol CP1
- R7: value 500 -> 470
- RV1: footprint Potentiometers:Potentiometer_Triwood_RM-065 -> Potentiometers:Potentiometer_Trimmer_Bourns_3214W
- RV2, RV3, RV4, RV5: footprint Potentiometers:Potentiometer_Bourns_3296W_3-8Zoll_Inline_ScrewUp -> Potentiometers:Potentiometer_Trimmer_Bourns_3296W
- RV6: footprint Potentiometers:Potentiometer_Trimmer_Bourns_3266W -> Potentiometers:Potentiometer_Trimmer_Bourns_3214W
- U2, U3: footprint anthoperso:SOP4 -> Librairie master:SOP4
Connections:
- net GND: now also P20.5 (P5), C10.2, C8.2; no longer P20.8 (P8)
- net RX_module: now also P20.8 (P8); no longer P20.4 (P4)
- net TX_module: now also P20.7 (P7); no longer P20.6 (P6)
- net VCC: now also P20.6 (P6), C10.1; no longer P20.7 (P7)
- net at C38.1, P26.1 (P1), U5.2 (VO): now also C8.1
- net at U3.4: now also P20.4 (P4); no longer P20.5 (P5)
Other:
- note added: "Switch"
- moved on the sheet: P17
