File: PCB LM386 amplifier/LM386Amplifier.kicad_pcb (KiCad board)
At the start: 2 copper layers, 36.8 x 25.4 mm, 21 parts, among them J1 JACK_2P, P1 CONN_01X02, P2 CONN_01X02, U1 LM386

Commit message: Update pcb files
Parts:
- moved RV2 5.08 mm to (137.8, 84.5), turned to 90 degrees
Routing:
- net (no net): track 0.00 -> 20.3 mm
- net Net-(R7-Pad1): track 8.78 -> 4.44 mm
- net Net-(R6-Pad1): track 7.51 -> 6.99 mm
Other:
- board size 36.8 x 25.4 mm -> 37.5 x 25.4 mm
- board text added: "+5V"
- board text added: "0"
- board text added: "A"
- board text added: "Ampli 2W"
- board text added: "B"
- board text added: "HP"
- board text added: "JACK"
- board text added: "©OpenAVRc"
