File: PCB Shield/Mega_2560 core mini_full_2.1_PM/OpenAVRc_Sticks.sch (KiCad schematic (older format))
At the start: 58 parts, among them P11 Trim, P12 Stick_left, P13 Stick_right, P14 Switch, P23 Rot_1, P24 Rot_2, P25 Keys, P28 5v/3,3v manches, P31 Pot2, P32 Pot1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

Commit message: Update pcb shield
Update core component (change pin 99 from GND to AGND).
Remove GND on AGND pin.
Parts:
- P33: footprint (none) -> Pin_Headers:Pin_Header_Straight_1x02_Pitch2.54mm
Changed lines of the file:
@@
 Sheet 2 7
 Title "Shield Mega2560 core Full"
-Date "2018-04-19"
+Date "2018-04-25"
 Rev "2.10"
 Comp "© Team OpenAVRc"
@@
 F 0 "P33" H 10450 1400 50  0000 C CNN
 F 1 "5V_CODERS" V 10550 1250 50  0000 C CNN
-F 2 "" H 10450 1250 50  0000 C CNN
+F 2 "Pin_Headers:Pin_Header_Straight_1x02_Pitch2.54mm" H 10450 1250 50  0001 C CNN
 F 3 "" H 10450 1250 50  0000 C CNN
 	1    10450 1250
