File: PCB Shield/Mega_2560 core mini_full_2.1_PM/OpenAVRc_Audio_Haptic.sch (KiCad schematic (older format))
At the start: 16 parts, among them P22 JQ6500_28P, P5 Vibreur, P8 Audio, Q2 MMBT2222ALT1

Commit message: Update schematic & pcb files
add mosfet function
Parts:
- removed D1, D2, D3: LL4148, Diodes_SMD:D_SOD-123, symbol MBR0520
- removed R1: 22K, Resistors_SMD:R_1206, symbol R-RESCUE-Mega_2560_core_mini_full_2.0
- removed R2: 1K, Resistors_SMD:R_1206, symbol R-RESCUE-Mega_2560_core_mini_full_2.0
- added D1, D2, D3: LL4148, Diodes_SMD:D_SOD-123, symbol DIODE
Connections:
- net Audio_Buzzer_out: now also P8.1 (P1)
- net JQ_Left_Out: now also P8.2 (P2)
- net VCC: now also D1.2 (K), D2.1 (A)
- net at C2.2, P5.1 (P1): now also D3.2 (K)
- net at C2.1, P5.2 (P2), Q2.3 (C): now also D1.1 (A)
- new net: D2.2 (K), D3.1 (A)
Other:
- moved on the sheet: C2, P5
Changed lines of the file:
@@
 Sheet 6 7
 Title "Shield Mega2560 core Full"
-Date "2018-03-06"
+Date "2018-03-16"
 Rev "2.10"
 Comp "© Team OpenAVRc"
@@
 L CONN_01X02 P5
 U 1 1 59C5A561
-P 10400 3500
-F 0 "P5" H 10400 3650 50  0000 C CNN
-F 1 "Vibreur" V 10500 3500 50  0000 C CNN
-F 2 "Pin_Headers:Pin_Header_Straight_1x02_Pitch2.54mm" H 10400 3500 50  0001 C CNN
-F 3 "" H 10400 3500 50  0000 C CNN
-	1    10400 3500
-	1    0    0    -1
-$EndComp
-$Comp
-L R-RESCUE-Mega_2560_core_mini_full_2.0 R1
-U 1 1 59C5A56F
-P 5900 3550
-F 0 "R1" V 5800 3550 50  0000 C CNN
-F 1 "22K" V 5900 3550 50  0000 C CNN
-F 2 "Resistors_SMD:R_1206" V 5830 3550 50  0001 C CNN
-F 3 "" H 5900 3550 50  0000 C CNN
-	1    5900 3550
-	1    0    0    -1
-$EndComp
-$Comp
-L R-RESCUE-Mega_2560_core_mini_full_2.0 R2
-U 1 1 59C5A576
-P 6000 3550
-F 0 "R2" V 6080 3550 50  0000 C CNN
-F 1 "1K" V 6000 3550 50  0000 C CNN
-F 2 "Resistors_SMD:R_1206" V 5930 3550 50  0001 C CNN
-F 3 "" H 6000 3550 50  0000 C CNN
-	1    6000 3550
+P 10650 3300
+F 0 "P5" H 10650 3450 50  0000 C CNN
+F 1 "Vibreur" V 10750 3300 50  0000 C CNN
+F 2 "Pin_Headers:Pin_Header_Straight_1x02_Pitch2.54mm" H 10650 3300 50  0001 C CNN
+F 3 "" H 10650 3300 50  0000 C CNN
+	1    10650 3300
 	1    0    0    -1
 $EndComp
@@
 $EndComp
 $Comp
-L MBR0520 D1
-U 1 1 59C5A5A7
-P 9050 3450
-F 0 "D1" H 9050 3550 50  0000 C CNN
-F 1 "LL4148" H 9050 3350 50  0000 C CNN
-F 2 "Diodes_SMD:D_SOD-123" H 9050 3275 50  0001 C CNN
-F 3 "" H 9050 3450 50  0001 C CNN
-	1    9050 3450
-	0    1    1    0
-$EndComp
-$Comp
 L R-RESCUE-Mega_2560_core_mini_full_2.0 R9
 U 1 1 59C5A5AE
@@
 L C-RESCUE-Mega_2560_core_mini_full_2.0 C2
 U 1 1 5A980AA9
-P 9950 3500
-F 0 "C2" H 9975 3600 50  0000 L CNN
-F 1 "100nF" H 10100 3500 50  0000 L CNN
-F 2 "Capacitors_SMD:C_1206" H 9988 3350 50  0001 C CNN
-F 3 "" H 9950 3500 50  0000 C CNN
-	1    9950 3500
-	-1   0    0    1
-$EndComp
-$Comp
-L MBR0520 D2
-U 1 1 5A980F3A
-P 9300 3250
-F 0 "D2" H 9300 3350 50  0000 C CNN
-F 1 "LL4148" H 9300 3150 50  0000 C CNN
-F 2 "Diodes_SMD:D_SOD-123" H 9300 3075 50  0001 C CNN
-F 3 "" H 9300 3250 50  0001 C CNN
-	1    9300 3250
-	-1   0    0    1
-$EndComp
-$Comp
-L MBR0520 D3
-U 1 1 5A980F85
-P 9700 3250
-F 0 "D3" H 9700 3350 50  0000 C CNN
-F 1 "LL4148" H 9700 3150 50  0000 C CNN
-F 2 "Diodes_SMD:D_SOD-123" H 9700 3075 50  0001 C CNN
-F 3 "" H 9700 3250 50  0001 C CNN
-	1    9700 3250
+P 10200 3300
+F 0 "C2" H 10225 3400 50  0000 L CNN
+F 1 "100nF" H 10350 3300 50  0000 L CNN
+F 2 "Capacitors_SMD:C_1206" H 10238 3150 50  0001 C CNN
+F 3 "" H 10200 3300 50  0000 C CNN
+	1    10200 3300
 	-1   0    0    1
 $EndComp
@@
 L VCC #PWR0110
 U 1 1 5A981097
-P 9050 3200
-F 0 "#PWR0110" H 9050 3050 50  0001 C CNN
-F 1 "VCC" H 9050 3350 50  0000 C CNN
-F 2 "" H 9050 3200 50  0000 C CNN
-F 3 "" H 9050 3200 50  0000 C CNN
-	1    9050 3200
+P 9050 3000
+F 0 "#PWR0110" H 9050 2850 50  0001 C CNN
+F 1 "VCC" H 9050 3150 50  0000 C CNN
+F 2 "" H 9050 3000 50  0000 C CNN
+F 3 "" H 9050 3000 50  0000 C CNN
+	1    9050 3000
 	1    0    0    -1
 $EndComp
@@
 	3500 4150 3350 4150
 Wire Wire Line
-	6000 3700 6000 4300
+	6000 3350 6000 4300
 Connection ~ 6200 3400
 Connection ~ 6500 3400
@@
 	6200 3250 6200 3750
 Wire Wire Line
-	5900 3700 5900 4300
+	5900 3350 5900 4300
 Wire Wire Line
 	4500 3050 5350 3050
@@
 	8250 3950 7950 3950
 Wire Wire Line
-	6000 3400 6000 3350
-Wire Wire Line
 	6000 3350 6100 3300
 Wire Wire Line
 	6100 3300 6100 3250
-Wire Wire Line
-	5900 3400 5900 3350
 Wire Wire Line
 	5900 3350 6000 3300
@@
 	9050 4150 9050 4400
 Wire Wire Line
-	9050 3200 9050 3300
-Wire Wire Line
-	9050 3750 9050 3600
-Wire Wire Line
-	9850 3250 10150 3250
-Wire Wire Line
-	9550 3250 9450 3250
-Wire Wire Line
-	9150 3250 9050 3250
-Connection ~ 9050 3250
-Wire Wire Line
-	10200 3450 10150 3450
-Wire Wire Line
-	10150 3450 10150 3250
-Wire Wire Line
-	9950 3350 9950 3250
-Connection ~ 9950 3250
-Wire Wire Line
-	10200 3550 10150 3550
-Wire Wire Line
-	10150 3550 10150 3700
-Wire Wire Line
-	10150 3700 9050 3700
+	9050 3000 9050 3200
+Wire Wire Line
+	9050 3600 9050 3750
+Wire Wire Line
+	10100 3050 10400 3050
+Wire Wire Line
+	9050 3050 9200 3050
+Connection ~ 9050 3050
+Wire Wire Line
+	10450 3250 10400 3250
+Wire Wire Line
+	10400 3250 10400 3050
+Wire Wire Line
+	10200 3150 10200 3050
+Connection ~ 10200 3050
+Wire Wire Line
+	10450 3350 10400 3350
+Wire Wire Line
+	10400 3350 10400 3700
+Wire Wire Line
+	10400 3700 9050 3700
 Connection ~ 9050 3700
 Wire Wire Line
-	9950 3650 9950 3700
-Connection ~ 9950 3700
+	10200 3450 10200 3700
+Connection ~ 10200 3700
+$Comp
+L DIODE D1
+U 1 1 5AABE17F
+P 9050 3400
+F 0 "D1" H 9050 3300 40  0000 C CNN
+F 1 "LL4148" H 9050 3500 40  0000 C CNN
+F 2 "Diodes_SMD:D_SOD-123" H 9050 3400 60  0001 C CNN
+F 3 "" H 9050 3400 60  0000 C CNN
+	1    9050 3400
+	0    -1   -1   0
+$EndComp
+$Comp
+L DIODE D2
+U 1 1 5AABE736
+P 9400 3050
+F 0 "D2" H 9400 2950 40  0000 C CNN
+F 1 "LL4148" H 9400 3150 40  0000 C CNN
+F 2 "Diodes_SMD:D_SOD-123" H 9400 3050 60  0001 C CNN
+F 3 "" H 9400 3050 60  0000 C CNN
+	1    9400 3050
+	1    0    0    -1
+$EndComp
+$Comp
+L DIODE D3
+U 1 1 5AABE7EC
+P 9900 3050
+F 0 "D3" H 9900 2950 40  0000 C CNN
+F 1 "LL4148" H 9900 3150 40  0000 C CNN
+F 2 "Diodes_SMD:D_SOD-123" H 9900 3050 60  0001 C CNN
+F 3 "" H 9900 3050 60  0000 C CNN
+	1    9900 3050
+	1    0    0    -1
+$EndComp
+Wire Wire Line
+	9700 3050 9600 3050
 $EndSCHEMATC

Commit message: Update pcb shield
Update core component (change pin 99 from GND to AGND).
Remove GND on AGND pin.
Parts:
- Q2: footprint SOT-23_MMBT2222 -> v2.1:SOT-23_MMBT2222
Changed lines of the file:
@@
 Sheet 6 7
 Title "Shield Mega2560 core Full"
-Date "2018-04-19"
+Date "2018-04-25"
 Rev "2.10"
 Comp "© Team OpenAVRc"
@@
 $EndDescr
 $Comp
-L GND-RESCUE-Mega_2560_core_mini_full_2.0 #PWR0101
+L GND-RESCUE-Mega_2560_core_mini_full_2.0 #PWR0100
 U 1 1 59C5A54C
 P 6500 3600
-F 0 "#PWR0101" H 6500 3350 50  0001 C CNN
+F 0 "#PWR0100" H 6500 3350 50  0001 C CNN
 F 1 "GND" H 6500 3450 50  0000 C CNN
 F 2 "" H 6500 3600 50  0000 C CNN
@@
 $EndComp
 $Comp
-L VCC #PWR0102
+L VCC #PWR0101
 U 1 1 59C5A552
 P 6200 3750
-F 0 "#PWR0102" H 6200 3600 50  0001 C CNN
+F 0 "#PWR0101" H 6200 3600 50  0001 C CNN
 F 1 "VCC" H 6200 3900 50  0000 C CNN
 F 2 "" H 6200 3750 50  0000 C CNN
@@
 $EndComp
 $Comp
-L VCC #PWR0103
+L VCC #PWR0102
 U 1 1 59C5A58E
 P 4000 4500
-F 0 "#PWR0103" H 4000 4350 50  0001 C CNN
+F 0 "#PWR0102" H 4000 4350 50  0001 C CNN
 F 1 "VCC" H 4000 4650 50  0000 C CNN
 F 2 "" H 4000 4500 50  0000 C CNN
@@
 $EndComp
 $Comp
-L GND-RESCUE-Mega_2560_core_mini_full_2.0 #PWR0104
+L GND-RESCUE-Mega_2560_core_mini_full_2.0 #PWR0103
 U 1 1 59C5A594
 P 3350 4400
-F 0 "#PWR0104" H 3350 4150 50  0001 C CNN
+F 0 "#PWR0103" H 3350 4150 50  0001 C CNN
 F 1 "GND" H 3350 4250 50  0000 C CNN
 F 2 "" H 3350 4400 50  0000 C CNN
@@
 $EndComp
 $Comp
-L GND-RESCUE-Mega_2560_core_mini_full_2.0 #PWR0105
+L GND-RESCUE-Mega_2560_core_mini_full_2.0 #PWR0104
 U 1 1 59C5A59A
 P 4650 4400
-F 0 "#PWR0105" H 4650 4150 50  0001 C CNN
+F 0 "#PWR0104" H 4650 4150 50  0001 C CNN
 F 1 "GND" H 4650 4250 50  0000 C CNN
 F 2 "" H 4650 4400 50  0000 C CNN
@@
 $EndComp
 $Comp
-L GND-RESCUE-Mega_2560_core_mini_full_2.0 #PWR0106
+L GND-RESCUE-Mega_2560_core_mini_full_2.0 #PWR0105
 U 1 1 59C5A5DF
 P 3650 4750
-F 0 "#PWR0106" H 3650 4500 50  0001 C CNN
+F 0 "#PWR0105" H 3650 4500 50  0001 C CNN
 F 1 "GND" H 3650 4600 50  0000 C CNN
 F 2 "" H 3650 4750 50  0000 C CNN
@@
 $EndComp
 $Comp
-L GND-RESCUE-Mega_2560_core_mini_full_2.0 #PWR0107
+L GND-RESCUE-Mega_2560_core_mini_full_2.0 #PWR0106
 U 1 1 59C5A5E5
 P 4300 4750
-F 0 "#PWR0107" H 4300 4500 50  0001 C CNN
+F 0 "#PWR0106" H 4300 4500 50  0001 C CNN
 F 1 "GND" H 4300 4600 50  0000 C CNN
 F 2 "" H 4300 4750 50  0000 C CNN
@@
 F 0 "Q2" H 9250 3850 50  0000 R CNN
 F 1 "MMBT2222ALT1" H 9700 3950 50  0000 R CNN
-F 2 "SOT-23_MMBT2222" H 8950 3950 60  0001 C CNN
+F 2 "v2.1:SOT-23_MMBT2222" H 8950 3950 60  0001 C CNN
 F 3 "" H 8950 3950 60  0000 C CNN
 	1    8950 3950
@@
 $EndComp
 $Comp
-L GND-RESCUE-Mega_2560_core_mini_full_2.0 #PWR0108
+L GND-RESCUE-Mega_2560_core_mini_full_2.0 #PWR0107
 U 1 1 5A9805CC
 P 9050 4400
-F 0 "#PWR0108" H 9050 4150 50  0001 C CNN
+F 0 "#PWR0107" H 9050 4150 50  0001 C CNN
 F 1 "GND" H 9050 4250 50  0000 C CNN
 F 2 "" H 9050 4400 50  0000 C CNN
@@
 $EndComp
 $Comp
-L VCC #PWR0109
+L VCC #PWR0108
 U 1 1 5A981097
 P 9050 3000
-F 0 "#PWR0109" H 9050 2850 50  0001 C CNN
+F 0 "#PWR0108" H 9050 2850 50  0001 C CNN
 F 1 "VCC" H 9050 3150 50  0000 C CNN
 F 2 "" H 9050 3000 50  0000 C CNN
