File: PCB/PCB A1335/A1335_Encodeur.sch (KiCad schematic (older format))
At the start: 13 parts, among them P1 CONN_01X04, Q1 MOS_N, Q2 MOS_N, U1 662K, U2 A1335LLETR-T

Commit message: A1335_upload_files
Parts:
- removed R3, R4, R5, R6: 0, R_1206, symbol R-RESCUE-Mega_2560_core_mini_full_2.0
- added W1, W2, W3, W4: 0, TESTPT, symbol TEST_2P
- C1, C2: footprint C_1206 -> C_0805_HandSoldering
- Q1, Q2: value MOS_N -> BSS138
- R1, R2: footprint R_1206 -> R_0805_HandSoldering
Connections:
- net GND: now also W1.2, W3.2
- net at C2.1, U2.2 (BYP): now also W2.2, W4.2
- net at U2.13 (SA0): now also W1.1, W2.1
- net at U2.12 (SA1): now also W3.1, W4.1
Changed lines of the file:
@@
 Sheet 1 1
 Title "Encodeur Angulaire Absolu A1335"
-Date "2018-11-29"
+Date "2018-12-01"
 Rev "0.1"
 Comp "OpenAVRc"
@@
 P 3900 3800
 F 0 "Q1" V 3800 4050 60  0000 R CNN
-F 1 "MOS_N" H 3910 3650 60  0001 R CNN
+F 1 "BSS138" V 4100 4000 60  0000 R CNN
 F 2 "SOT-23_MOS_P" H 3900 3800 60  0001 C CNN
 F 3 "" H 3900 3800 60  0000 C CNN
@@
 P 3900 4600
 F 0 "Q2" V 3750 4850 60  0000 R CNN
-F 1 "MOS_N" H 3910 4450 60  0001 R CNN
+F 1 "BSS138" V 4100 4800 60  0000 R CNN
 F 2 "SOT-23_MOS_P" H 3900 4600 60  0001 C CNN
 F 3 "" H 3900 4600 60  0000 C CNN
@@
 F 0 "R1" V 4430 3950 50  0000 C CNN
 F 1 "10K" V 4350 3950 50  0000 C CNN
-F 2 "R_1206" V 4280 3950 50  0001 C CNN
+F 2 "R_0805_HandSoldering" V 4280 3950 50  0001 C CNN
 F 3 "" H 4350 3950 50  0000 C CNN
 	1    4350 3950
@@
 F 0 "R2" V 4430 4750 50  0000 C CNN
 F 1 "10K" V 4350 4750 50  0000 C CNN
-F 2 "R_1206" V 4280 4750 50  0001 C CNN
+F 2 "R_0805_HandSoldering" V 4280 4750 50  0001 C CNN
 F 3 "" H 4350 4750 50  0000 C CNN
 	1    4350 4750
@@
 Connection ~ 4350 5000
 $Comp
-L +3,3V #PWR6
+L +3,3V #PWR01
 U 1 1 5BFBC0F5
 P 4500 4200
-F 0 "#PWR6" H 4500 4160 30  0001 C CNN
+F 0 "#PWR01" H 4500 4160 30  0001 C CNN
 F 1 "+3,3V" H 4500 4310 30  0000 C CNN
 F 2 "" H 4500 4200 60  0001 C CNN
@@
 $EndComp
 $Comp
-L +3,3V #PWR7
+L +3,3V #PWR02
 U 1 1 5BFBC113
 P 4500 5000
-F 0 "#PWR7" H 4500 4960 30  0001 C CNN
+F 0 "#PWR02" H 4500 4960 30  0001 C CNN
 F 1 "+3,3V" H 4500 5110 30  0000 C CNN
 F 2 "" H 4500 5000 60  0001 C CNN
@@
 $EndComp
 $Comp
-L +3,3V #PWR8
+L +3,3V #PWR03
 U 1 1 5BFBC14F
 P 4600 2800
-F 0 "#PWR8" H 4600 2760 30  0001 C CNN
+F 0 "#PWR03" H 4600 2760 30  0001 C CNN
 F 1 "+3,3V" H 4600 2910 30  0000 C CNN
 F 2 "" H 4600 2800 60  0001 C CNN
@@
 	3950 3100 3950 3250
 $Comp
-L +5V #PWR3
+L +5V #PWR04
 U 1 1 5BFBC1B5
 P 3250 2800
-F 0 "#PWR3" H 3250 2890 20  0001 C CNN
+F 0 "#PWR04" H 3250 2890 20  0001 C CNN
 F 1 "+5V" H 3250 2890 30  0000 C CNN
 F 2 "" H 3250 2800 60  0001 C CNN
@@
 $EndComp
 $Comp
-L GND #PWR4
+L GND #PWR05
 U 1 1 5BFBC1D3
 P 3950 3250
-F 0 "#PWR4" H 3950 3250 30  0001 C CNN
+F 0 "#PWR05" H 3950 3250 30  0001 C CNN
 F 1 "GND" H 3950 3180 30  0001 C CNN
 F 2 "" H 3950 3250 60  0001 C CNN
@@
 	6300 3400 6000 3400
 $Comp
-L +5V #PWR9
+L +5V #PWR06
 U 1 1 5BFBC450
 P 6000 3400
-F 0 "#PWR9" H 6000 3490 20  0001 C CNN
+F 0 "#PWR06" H 6000 3490 20  0001 C CNN
 F 1 "+5V" H 6000 3490 30  0000 C CNN
 F 2 "" H 6000 3400 60  0001 C CNN
@@
 Connection ~ 6650 4250
 $Comp
-L GND #PWR10
+L GND #PWR07
 U 1 1 5BFBC534
 P 6650 4300
-F 0 "#PWR10" H 6650 4300 30  0001 C CNN
+F 0 "#PWR07" H 6650 4300 30  0001 C CNN
 F 1 "GND" H 6650 4230 30  0001 C CNN
 F 2 "" H 6650 4300 60  0001 C CNN
@@
 $EndComp
 $Comp
-L GND #PWR11
+L GND #PWR08
 U 1 1 5BFBC57B
 P 6950 4300
-F 0 "#PWR11" H 6950 4300 30  0001 C CNN
+F 0 "#PWR08" H 6950 4300 30  0001 C CNN
 F 1 "GND" H 6950 4230 30  0001 C CNN
 F 2 "" H 6950 4300 60  0001 C CNN
@@
 F 0 "C1" H 4500 3200 40  0000 L CNN
 F 1 "100nF" H 4506 3015 40  0000 L CNN
-F 2 "C_1206" H 4538 2950 30  0001 C CNN
+F 2 "C_0805_HandSoldering" H 4538 2950 30  0001 C CNN
 F 3 "" H 4500 3100 60  0000 C CNN
 	1    4500 3100
@@
 	4500 3300 4500 3400
 $Comp
-L GND #PWR5
+L GND #PWR09
 U 1 1 5BFBC83C
 P 4500 3400
-F 0 "#PWR5" H 4500 3400 30  0001 C CNN
+F 0 "#PWR09" H 4500 3400 30  0001 C CNN
 F 1 "GND" H 4500 3330 30  0001 C CNN
 F 2 "" H 4500 3400 60  0001 C CNN
@@
 	1    0    0    -1
 $EndComp
-$Comp
-L R-RESCUE-Mega_2560_core_mini_full_2.0 R4
-U 1 1 5BFBC942
-P 7650 3600
-F 0 "R4" V 7600 3750 50  0000 C CNN
-F 1 "0" V 7650 3600 50  0000 C CNN
-F 2 "R_1206" V 7580 3600 50  0001 C CNN
-F 3 "" H 7650 3600 50  0000 C CNN
-	1    7650 3600
-	0    1    1    0
-$EndComp
-$Comp
-L R-RESCUE-Mega_2560_core_mini_full_2.0 R3
-U 1 1 5BFBCA52
-P 7650 3500
-F 0 "R3" V 7600 3650 50  0000 C CNN
-F 1 "0" V 7650 3500 50  0000 C CNN
-F 2 "R_1206" V 7580 3500 50  0001 C CNN
-F 3 "" H 7650 3500 50  0000 C CNN
-	1    7650 3500
-	0    1    1    0
-$EndComp
-$Comp
-L R-RESCUE-Mega_2560_core_mini_full_2.0 R5
-U 1 1 5BFBCA7D
-P 7650 3700
-F 0 "R5" V 7600 3850 50  0000 C CNN
-F 1 "0" V 7650 3700 50  0000 C CNN
-F 2 "R_1206" V 7580 3700 50  0001 C CNN
-F 3 "" H 7650 3700 50  0000 C CNN
-	1    7650 3700
-	0    1    1    0
-$EndComp
-$Comp
-L R-RESCUE-Mega_2560_core_mini_full_2.0 R6
-U 1 1 5BFBCABD
-P 7650 3800
-F 0 "R6" V 7600 3950 50  0000 C CNN
-F 1 "0" V 7650 3800 50  0000 C CNN
-F 2 "R_1206" V 7580 3800 50  0001 C CNN
-F 3 "" H 7650 3800 50  0000 C CNN
-	1    7650 3800
-	0    1    1    0
-$EndComp
-Wire Wire Line
-	7300 3600 7500 3600
-Wire Wire Line
-	7450 3600 7450 3500
-Wire Wire Line
-	7450 3500 7500 3500
-Connection ~ 7450 3600
-Wire Wire Line
-	7300 3700 7500 3700
-Wire Wire Line
-	7500 3800 7450 3800
-Wire Wire Line
-	7450 3800 7450 3700
-Connection ~ 7450 3700
-Wire Wire Line
-	7800 3500 7900 3500
 Wire Wire Line
 	7900 3500 7900 3900
 Wire Wire Line
-	7800 3700 7900 3700
-Connection ~ 7900 3700
-Wire Wire Line
-	8000 3800 7800 3800
-Wire Wire Line
 	8000 3400 8000 3800
-Wire Wire Line
-	8000 3600 7800 3600
 Connection ~ 8000 3600
 Wire Wire Line
 	7300 3400 8200 3400
 $Comp
-L GND #PWR12
+L GND #PWR010
 U 1 1 5BFBCE12
 P 7900 3900
-F 0 "#PWR12" H 7900 3900 30  0001 C CNN
+F 0 "#PWR010" H 7900 3900 30  0001 C CNN
 F 1 "GND" H 7900 3830 30  0001 C CNN
 F 2 "" H 7900 3900 60  0001 C CNN
@@
 F 0 "C2" H 8200 3750 40  0000 L CNN
 F 1 "100nF" H 8206 3565 40  0000 L CNN
-F 2 "C_1206" H 8238 3500 30  0001 C CNN
+F 2 "C_0805_HandSoldering" H 8238 3500 30  0001 C CNN
 F 3 "" H 8200 3650 60  0000 C CNN
 	1    8200 3650
@@
 $EndComp
 $Comp
-L GND #PWR13
+L GND #PWR011
 U 1 1 5BFBCFC6
 P 8200 3900
-F 0 "#PWR13" H 8200 3900 30  0001 C CNN
+F 0 "#PWR011" H 8200 3900 30  0001 C CNN
 F 1 "GND" H 8200 3830 30  0001 C CNN
 F 2 "" H 8200 3900 60  0001 C CNN
@@
 	1250 3950 1900 3950
 $Comp
-L GND #PWR1
+L GND #PWR012
 U 1 1 5BFFB77C
 P 1900 4150
-F 0 "#PWR1" H 1900 4150 30  0001 C CNN
+F 0 "#PWR012" H 1900 4150 30  0001 C CNN
 F 1 "GND" H 1900 4080 30  0001 C CNN
 F 2 "" H 1900 4150 60  0001 C CNN
@@
 $EndComp
 $Comp
-L +5V #PWR2
+L +5V #PWR013
 U 1 1 5BFFB7AE
 P 1900 4250
-F 0 "#PWR2" H 1900 4340 20  0001 C CNN
+F 0 "#PWR013" H 1900 4340 20  0001 C CNN
 F 1 "+5V" H 1900 4340 30  0000 C CNN
 F 2 "" H 1900 4250 60  0001 C CNN
@@
 	1    0    0    -1
 $EndComp
+$Comp
+L TEST_2P W1
+U 1 1 5C0234C6
+P 7600 3500
+F 0 "W1" H 7750 3550 50  0000 C CNN
+F 1 "0" H 7600 3430 50  0001 C CNN
+F 2 "TESTPT" H 7600 3500 50  0001 C CNN
+F 3 "" H 7600 3500 50  0000 C CNN
+	1    7600 3500
+	1    0    0    -1
+$EndComp
+$Comp
+L TEST_2P W2
+U 1 1 5C02380C
+P 7600 3600
+F 0 "W2" H 7750 3650 50  0000 C CNN
+F 1 "0" H 7600 3530 50  0001 C CNN
+F 2 "TESTPT" H 7600 3600 50  0001 C CNN
+F 3 "" H 7600 3600 50  0000 C CNN
+	1    7600 3600
+	1    0    0    -1
+$EndComp
+$Comp
+L TEST_2P W3
+U 1 1 5C0238AE
+P 7600 3700
+F 0 "W3" H 7750 3750 50  0000 C CNN
+F 1 "0" H 7600 3630 50  0001 C CNN
+F 2 "TESTPT" H 7600 3700 50  0001 C CNN
+F 3 "" H 7600 3700 50  0000 C CNN
+	1    7600 3700
+	1    0    0    -1
+$EndComp
+$Comp
+L TEST_2P W4
+U 1 1 5C0238E2
+P 7600 3800
+F 0 "W4" H 7750 3850 50  0000 C CNN
+F 1 "0" H 7600 3730 50  0001 C CNN
+F 2 "TESTPT" H 7600 3800 50  0001 C CNN
+F 3 "" H 7600 3800 50  0000 C CNN
+	1    7600 3800
+	1    0    0    -1
+$EndComp
+Wire Wire Line
+	7800 3500 7900 3500
+Wire Wire Line
+	7800 3700 7900 3700
+Connection ~ 7900 3700
+Wire Wire Line
+	8000 3800 7800 3800
+Wire Wire Line
+	7800 3600 8000 3600
+Wire Wire Line
+	7400 3600 7300 3600
+Wire Wire Line
+	7350 3600 7350 3500
+Wire Wire Line
+	7350 3500 7400 3500
+Connection ~ 7350 3600
+Wire Wire Line
+	7400 3700 7300 3700
+Wire Wire Line
+	7400 3800 7350 3800
+Wire Wire Line
+	7350 3800 7350 3700
+Connection ~ 7350 3700
 $EndSCHEMATC
