File: PCB/PCB Multiswitch 8/MutltiSwitch_Sw8.sch (KiCad schematic (older format))
At the start: 10 parts, among them IC1 ATTINY84-P, IC2 ULN2803, P1 OUTPUT_1-8, P8 XANY_INPUT, X1 16Mhz

Commit message: Update_PCB-Multiswitch_8
Parts:
- removed P1: OUTPUT_1-8, Pin_Header_Straight_1x09_Pitch2.54mm, symbol CONN_01X09
- added D2: LL4148, D_SOD-123, symbol DIODE
- added P1: +V=VRx / +V<VRx, Pin_Header_Straight_1x03_Pitch2.54mm, symbol CONN_01X03
- added P3: SERVO, Pin_Header_Straight_1x03_Pitch2.54mm, symbol CONN_01X03
- added P4: SEL_ALIM, Pin_Header_Straight_1x03_Pitch2.54mm, symbol CONN_01X03
- added P5: OUTPUT_1X8, Pin_Header_Straight_1x09_Pitch2.54mm, symbol CONN_01X08
- added P6: VExt, Faston_V-5_08, symbol CONN_01X02
- added P7: OUTPUT_1X8_ALIM, Pin_Header_Straight_1x09_Pitch2.54mm, symbol CONN_01X08
- added R1: 1K, R_1206, symbol R
- R2: value 470 -> 330
- renumbered P8 to P2
Connections:
- net +5V: now also D1.1 (A), D2.2 (K), P1.2 (P2), P1.3 (P3), P3.2 (P2); no longer P2.2 (P2)
- net GND: now also P3.3 (P3), P6.1 (P1); no longer D1.2 (K)
- net at IC2.10 (COM): now also P4.1 (P1)
- net at IC2.11 (O8): now also P5.8 (P8)
- net at IC2.12 (O7): now also P5.7 (P7)
- net at IC2.13 (O6): now also P5.6 (P6)
- net at IC2.14 (O5): now also P5.5 (P5)
- net at IC2.15 (O4): now also P5.4 (P4)
- net at IC2.16 (O3): now also P5.3 (P3)
- net at IC2.17 (O2): now also P5.2 (P2)
- net at IC2.18 (O1): now also P5.1 (P1)
- net at P2.1 (P1): now also R1.1; no longer IC1.5 ((PCINT10/CKOUT/OC0A/INT0)PB2)
- net at IC1.4 ((PCINT11/dW/~RESET~)PB3), R2.1: now also P3.1 (P1)
- net at R2.2: now also D1.2 (K); no longer D1.1 (A)
- new net: IC1.5 ((PCINT10/CKOUT/OC0A/INT0)PB2), R1.2
- new net: P4.2 (P2), P4.3 (P3), P6.2 (P2), P7.1 (P1), P7.2 (P2), P7.3 (P3), P7.4 (P4), P7.5 (P5), P7.6 (P6), P7.7 (P7), P7.8 (P8)
- new net +6V: D2.1 (A), P1.1 (P1), P2.2 (P2)
Other:
- moved on the sheet: C1, C2, C3, D1, IC1, IC2, P2, R2, X1
