File: PCB/MutltiSwitch_Sw16/MutltiSwitch_Sw16.sch (KiCad schematic (older format))
At the start: 39 parts, among them IC1 ATMEGA328-P, P1 OUTPUT_9-16, P10 FTDI, P11 ICSP, P12 5v/6v, P13 DIODE2, P14 DIODE1, P15 SERVO, P16 GND_EXT, P17 ALIM_EXT2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

Commit message: Update_PCB_Multiswitch_16
Parts:
- removed P1: OUTPUT_9-16, symbol CONN_01X09
- removed P12: 5v/6v, symbol CONN_01X02
- removed P13: DIODE2, symbol CONN_01X02
- removed P14: DIODE1, symbol CONN_01X02
- removed P2: OUTPUT_9-16_ALIM, symbol CONN_01X09
- removed P4: OUTPUT_1-8, symbol CONN_01X09
- removed P5: OUTPUT_1-8_ALIM, symbol CONN_01X09
- removed P9: OUTPUT_1-8_GND, symbol CONN_01X09
- added D3: LL4148, mylib:D_SOD-123, symbol DIODE
- added P1: OUTPUT_9-16, mylib:Pin_Header_Straight_1x08_Pitch2.54mm, symbol CONN_01X08
- added P12: +V = VRx / +V < VRx, mylib:Pin_Header_Straight_1x03_Pitch2.54mm, symbol CONN_01X03
- added P13: DIODE2, mylib:Pin_Header_Straight_1x03_Pitch2.54mm, symbol CONN_01X03
- added P14: DIODE1, mylib:Pin_Header_Straight_1x03_Pitch2.54mm, symbol CONN_01X03
- added P2: OUTPUT_9-16_ALIM, mylib:Pin_Header_Straight_1x08_Pitch2.54mm, symbol CONN_01X08
- added P4: OUTPUT_1-8, mylib:Pin_Header_Straight_1x08_Pitch2.54mm, symbol CONN_01X08
- added P5: OUTPUT_1-8_ALIM, mylib:Pin_Header_Straight_1x08_Pitch2.54mm, symbol CONN_01X08
- added P9: OUTPUT_1-8_GND, mylib:Pin_Header_Straight_1x08_Pitch2.54mm, symbol CONN_01X08
- C1, C2, C3, C4, C5: footprint (none) -> mylib:C_1206
- D1: footprint (none) -> mylib:LED_1206
- D2: value 1N4001 -> LL4148; footprint (none) -> mylib:D_SOD-123
- IC1: footprint (none) -> mylib:DIP-28_W7.62mm_LongPads
- P10, P11: footprint (none) -> mylib:Pin_Header_Straight_2x03_Pitch2.54mm
- P16: footprint Faston_V-5_08 -> mylib:Faston_V-5_08
- P17: value ALIM_EXT2 -> VExt2; footprint Faston_V-5_08 -> mylib:Faston_V-5_08
- P3: value SELECT_ALIM2 -> SEL_ALIM2; footprint (none) -> mylib:Pin_Header_Straight_1x03_Pitch2.54mm
- P6: value SELECT_ALIM1 -> SEL_ALIM1; footprint (none) -> mylib:Pin_Header_Straight_1x03_Pitch2.54mm
- P7: value ALIM_EXT1 -> VExt1; footprint Faston_V-5_08 -> mylib:Faston_V-5_08
- P8: footprint (none) -> mylib:Pin_Header_Straight_1x03_Pitch2.54mm
- R1, R10, R11, R3, R4, R5, R6, R7, R8, R9: footprint (none) -> mylib:R_1206
- R2: value 10K -> 330; footprint (none) -> mylib:R_1206
- U1, U2: footprint (none) -> mylib:DIP-18_W7.62mm_LongPads
- X1: footprint (none) -> mylib:HC-39
Connections:
- wire segments 190 -> 196
Other:
- note added: "- Load +"
- note added: "Servo"
- note added: "Signal + -"
- moved on the sheet: C1, C2, C3, C4, C5, D1, D2, IC1, P10, P11, P15, P16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

Commit message: Update_PCB_multiswitch_16
Parts:
- added R12: 10K, mylib:R_1206, symbol R
- added R13: 1M, mylib:R_1206, symbol R
- C2, C4: value 100nF -> 22pF
Connections:
- net +5V: now also R12.1; no longer D1.1 (A), P15.2 (P2), P3.1 (P1), P6.1 (P1)
- net GND: now also D1.2 (K)
- net at C2.1, IC1.10 ((PCINT7/XTAL2/TOSC2)PB7), X1.2: now also R13.2
- net at IC1.2 ((PCINT16/RXD)PD0), P10.3 (P3): now also R12.2
- net at C4.1, IC1.9 ((PCINT6/XTAL1/TOSC1)PB6), X1.1: now also R13.1
- net at R2.2: now also D1.1 (A); no longer D1.2 (K)
- net +6V renamed +VRx
- net +VRx: now also P15.2 (P2), P3.1 (P1), P6.1 (P1)
