File: PCB/MutltiSwitch_Sw16/MutltiSwitch_Sw16.kicad_pcb (KiCad board)
At the start: 2 copper layers, 43 parts, among them IC1 ATMEGA328-P, P1 OUTPUT_9-16, P10 FTDI, P11 ICSP, P12 5v/6v, P13 DIODE2, P14 DIODE1, P15 SERVO, P16 GND_EXT, P17 ALIM_EXT2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

Commit message: Update_PCB_Multiswitch_16
Parts:
- added D3: LL4148, mylib:D_SOD-123, B.Cu at (145.9, 78.9)
- C1, C2, C3, C4, C5: footprint C_1206 -> mylib:C_1206
- D1: footprint LED_1206 -> mylib:LED_1206
- D2: value 1N4001 -> LL4148; footprint D_DO-204AC -> mylib:D_SOD-123
- IC1: footprint DIP-28_W7.62mm_LongPads -> mylib:DIP-28_W7.62mm_LongPads
- P1, P2, P4, P5, P9: footprint Pin_Header_Straight_1x09_Pitch2.54mm -> mylib:Pin_Header_Straight_1x08_Pitch2.54mm
- P10, P11: footprint Pin_Header_Straight_2x03_Pitch2.54mm -> mylib:Pin_Header_Straight_2x03_Pitch2.54mm
- P12: value 5v/6v -> +V = VRx / +V < VRx; footprint Pin_Header_Straight_1x02_Pitch2.54mm -> mylib:Pin_Header_Straight_1x03_Pitch2.54mm
- P13, P14: footprint Pin_Header_Straight_1x02_Pitch2.54mm -> mylib:Pin_Header_Straight_1x03_Pitch2.54mm
- P16: footprint Faston_V-5_08 -> mylib:Faston_V-5_08
- P17: value ALIM_EXT2 -> VExt2; footprint Faston_V-5_08 -> mylib:Faston_V-5_08
- P3: value SELECT_ALIM2 -> SEL_ALIM2; footprint Pin_Header_Straight_1x03_Pitch2.54mm -> mylib:Pin_Header_Straight_1x03_Pitch2.54mm
- P6: value SELECT_ALIM1 -> SEL_ALIM1; footprint Pin_Header_Straight_1x03_Pitch2.54mm -> mylib:Pin_Header_Straight_1x03_Pitch2.54mm
- P7: value ALIM_EXT1 -> VExt1; footprint Faston_V-5_08 -> mylib:Faston_V-5_08
- P8: footprint Pin_Header_Straight_1x03_Pitch2.54mm -> mylib:Pin_Header_Straight_1x03_Pitch2.54mm
- R1, R10, R11, R3, R4, R5, R6, R7, R8, R9: footprint R_1206 -> mylib:R_1206
- R2: value 10K -> 330; footprint R_1206 -> mylib:R_1206
- U1, U2: footprint DIP-18_W7.62mm_LongPads -> mylib:DIP-18_W7.62mm_LongPads
- X1: footprint HC-39 -> mylib:HC-39
- moved D2 3.59 mm to (158.1, 104.1)
- moved P12 1.27 mm to (156.8, 101.6)
Connections:
- P11 pad 5: Net-(C5-Pad2) -> Net-(C5-Pad1)
- P13 pad 2: Net-(P1-Pad9) -> Net-(P13-Pad2)
- P2 pad 1: Net-(P1-Pad9) -> Net-(P13-Pad2)
- P2 pad 2: Net-(P1-Pad9) -> Net-(P13-Pad2)
- P2 pad 3: Net-(P1-Pad9) -> Net-(P13-Pad2)
- P2 pad 4: Net-(P1-Pad9) -> Net-(P13-Pad2)
- P2 pad 5: Net-(P1-Pad9) -> Net-(P13-Pad2)
- P2 pad 6: Net-(P1-Pad9) -> Net-(P13-Pad2)
- P2 pad 7: Net-(P1-Pad9) -> Net-(P13-Pad2)
- P2 pad 8: Net-(P1-Pad9) -> Net-(P13-Pad2)
- P3 pad 2: Net-(P1-Pad9) -> Net-(P13-Pad2)
Routing:
- net Net-(C5-Pad1): track 6.95 -> 75.5 mm
- net Net-(C5-Pad2): track 80.6 -> 16.9 mm
- net Net-(P1-Pad9): track 30.7 -> 0.00 mm
- net Net-(P13-Pad2): track 0.00 -> 30.7 mm
- net +5V: track 113.0 -> 106.0 mm
Other:
- board outline added: 63.5 x 41.9 mm
- board text added: "8x10K"
- board text added: "@ OpenAVRc Team"
- board text added: "MS16 X-Any"
- board text removed: "8x1K"
- board text removed: "@ OpenAVRC Team"
- board text removed: "Ms16 X-Any"

Commit message: Update_PCB_multiswitch_16
Parts:
- added R12: 10K, mylib:R_1206, B.Cu at (137.8, 79.8)
- added R13: 1M, mylib:R_1206, B.Cu at (139.4, 95.4)
- C2, C4: value 100nF -> 22pF
- moved P11 2.67 mm to (173.6, 101.5)
- turned R2 to 270 degrees
Connections:
- D1 pad 1: +5V -> Net-(D1-Pad1)
- D1 pad 2: Net-(D1-Pad2) -> GND
- D2 pad 1: +6V -> +VRx
- P12 pad 2: +6V -> +VRx
- P12 pad 3: +6V -> +VRx
- P15 pad 2: +5V -> +VRx
- P3 pad 1: +5V -> +VRx
- P6 pad 1: +5V -> +VRx
- P8 pad 2: +6V -> +VRx
- R2 pad 2: Net-(D1-Pad2) -> Net-(D1-Pad1)
Routing:
- net +VRx: track 0.00 -> 36.8 mm
- net +6V: track 13.1 -> 0.00 mm
- net +5V: track 106.0 -> 93.7 mm, vias 0 -> 2
- net Net-(IC1-Pad18): track 49.5 -> 42.7 mm, vias 1 -> 0
- net Net-(D1-Pad1): track 0.00 -> 3.61 mm, vias 0 -> 1
- net Net-(IC1-Pad19): track 86.4 -> 83.2 mm
- net Net-(D1-Pad2): track 3.10 -> 0.00 mm, vias 1 -> 0
- net Net-(C5-Pad1): track 75.5 -> 72.9 mm
- net Net-(IC1-Pad28): track 46.8 -> 44.5 mm
- net Net-(IC1-Pad17): track 39.4 -> 37.6 mm
- net GND: track 8.73 -> 10.4 mm, vias 0 -> 1
- net Net-(IC1-Pad2): track 12.6 -> 14.2 mm

Commit message: Update_PCB_Multiswitch_16
Other:
- board text added: "VExt1"
- board text added: "VExt2"
- board text added: "VExt_GND"
Changed lines of the file:
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@@
     (links 135)
     (no_connects 0)
-    (area 133.274999 69.774999 196.925001 111.835001)
+    (area 128.127857 67.495 207.239999 117.000001)
     (thickness 1.6)
-    (drawings 22)
+    (drawings 25)
     (tracks 334)
     (zones 0)
@@
   )
   (layers
-    (0 F.Cu signal)
+    (0 F.Cu signal hide)
     (31 B.Cu signal)
     (32 B.Adhes user hide)
@@
     (34 B.Paste user hide)
     (35 F.Paste user hide)
-    (36 B.SilkS user hide)
+    (36 B.SilkS user)
     (37 F.SilkS user hide)
     (38 B.Mask user hide)
@@
     (46 B.CrtYd user hide)
     (47 F.CrtYd user hide)
-    (48 B.Fab user hide)
-    (49 F.Fab user)
+    (48 B.Fab user)
+    (49 F.Fab user hide)
   )
   (setup
@@
     (aux_axis_origin 133.35 111.76)
     (grid_origin 133.35 111.76)
-    (visible_elements 7FFDFFFF)
+    (visible_elements 7FFFFDDF)
     (pcbplotparams
       (layerselection 0x10000_00000000)
       (usegerberextensions false)
-      (excludeedgelayer false)
+      (excludeedgelayer true)
       (linewidth 0.100000)
       (plotframeref false)
@@
       (subtractmaskfromsilk false)
       (outputformat 4)
-      (mirror true)
+      (mirror false)
       (drillshape 0)
       (scaleselection 1)
@@
       (effects (font (size 1 1) (thickness 0.15)) (justify mirror))
     )
-    (fp_text value LL4148 (at 0.127 1.778 180) (layer B.Fab)
-      (effects (font (size 1 1) (thickness 0.15)) (justify mirror))
-    )
-    (fp_text user %R (at 0.127 3.429 180) (layer B.Fab)
+    (fp_text value LL4148 (at 1.397 -1.905 180) (layer B.Fab)
+      (effects (font (size 1 1) (thickness 0.15)) (justify mirror))
+    )
+    (fp_text user %R (at -3.556 0 180) (layer B.Fab)
       (effects (font (size 1 1) (thickness 0.15)) (justify mirror))
     )
@@
     (descr "Through hole straight pin header, 1x03, 2.54mm pitch, single row")
     (tags "Through hole pin header THT 1x03 2.54mm single row")
-    (fp_text reference P13 (at 0 7.493 270) (layer F.SilkS)
+    (fp_text reference P13 (at 2.286 3.429 360) (layer F.SilkS)
       (effects (font (size 1 1) (thickness 0.15)))
     )
@@
     (descr "Through hole straight pin header, 1x03, 2.54mm pitch, single row")
     (tags "Through hole pin header THT 1x03 2.54mm single row")
-    (fp_text reference P14 (at 0 7.493 270) (layer F.SilkS)
+    (fp_text reference P14 (at 2.159 2.921 360) (layer F.SilkS)
       (effects (font (size 1 1) (thickness 0.15)))
     )
@@
     (descr "Through hole straight pin header, 1x03, 2.54mm pitch, single row")
     (tags "Through hole pin header THT 1x03 2.54mm single row")
-    (fp_text reference P15 (at 0.127 -2.286 270) (layer F.SilkS)
+    (fp_text reference P15 (at 2.159 5.207 360) (layer F.SilkS)
       (effects (font (size 1 1) (thickness 0.15)))
     )
@@
     (descr "Through hole straight pin header, 2x03, 2.54mm pitch, double rows")
     (tags "Through hole pin header THT 2x03 2.54mm double row")
-    (fp_text reference P11 (at 4.826 2.794 180) (layer F.SilkS)
+    (fp_text reference P11 (at -2.286 2.921 180) (layer F.SilkS)
       (effects (font (size 1 1) (thickness 0.15)))
     )
@@
     (tags "resistor 1206")
     (attr smd)
-    (fp_text reference R2 (at 0 1.85 270) (layer B.SilkS)
-      (effects (font (size 1 1) (thickness 0.15)) (justify mirror))
-    )
-    (fp_text value 330 (at 0 -1.95 270) (layer B.Fab)
+    (fp_text reference R2 (at 0 1.651 270) (layer B.SilkS)
+      (effects (font (size 1 1) (thickness 0.15)) (justify mirror))
+    )
+    (fp_text value 330 (at 0.127 1.651 270) (layer B.Fab)
       (effects (font (size 1 1) (thickness 0.15)) (justify mirror))
     )
@@
     (descr "Through hole straight pin header, 1x09, 2.54mm pitch, single row")
     (tags "Through hole pin header THT 1x09 2.54mm single row")
-    (fp_text reference P1 (at 0.127 -1.778) (layer F.SilkS)
+    (fp_text reference P1 (at 0.127 -2.413) (layer F.SilkS)
       (effects (font (size 1 1) (thickness 0.15)))
     )
@@
     (descr "Through hole straight pin header, 1x09, 2.54mm pitch, single row")
     (tags "Through hole pin header THT 1x09 2.54mm single row")
-    (fp_text reference P2 (at 0 -1.778) (layer F.SilkS)
+    (fp_text reference P2 (at 0 -2.413) (layer F.SilkS)
       (effects (font (size 1 1) (thickness 0.15)))
     )
@@
     (descr "Through hole straight pin header, 1x09, 2.54mm pitch, single row")
     (tags "Through hole pin header THT 1x09 2.54mm single row")
-    (fp_text reference P4 (at 0 -1.778) (layer F.SilkS)
+    (fp_text reference P4 (at 0 -2.286) (layer F.SilkS)
       (effects (font (size 1 1) (thickness 0.15)))
     )
@@
     (descr "Through hole straight pin header, 1x09, 2.54mm pitch, single row")
     (tags "Through hole pin header THT 1x09 2.54mm single row")
-    (fp_text reference P5 (at 0 -1.778) (layer F.SilkS)
+    (fp_text reference P5 (at 0 -2.286) (layer F.SilkS)
       (effects (font (size 1 1) (thickness 0.15)))
     )
@@
     (descr "Through hole straight pin header, 1x09, 2.54mm pitch, single row")
     (tags "Through hole pin header THT 1x09 2.54mm single row")
-    (fp_text reference P9 (at 0 -1.778) (layer F.SilkS)
+    (fp_text reference P9 (at 0 -2.286) (layer F.SilkS)
       (effects (font (size 1 1) (thickness 0.15)))
     )
@@
     )
   )
+  (gr_text VExt_GND (at 190.754 98.679 90) (layer F.SilkS)
+    (effects (font (size 1 1) (thickness 0.15)))
+  )
+  (gr_text VExt1 (at 172.72 105.537) (layer F.SilkS)
+    (effects (font (size 1 1) (thickness 0.15)))
+  )
+  (gr_text VExt2 (at 184.277 105.791) (layer F.SilkS)
+    (effects (font (size 1 1) (thickness 0.15)))
+  )
   (gr_line (start 196.85 69.85) (end 196.85 111.76) (angle 90) (layer Edge.Cuts) (width 0.15))
