File: PCB/MutltiSwitch_Sw8/MutltiSwitch_Sw8.sch (KiCad schematic (older format))
At the start: 32 parts, among them IC1 ATTINY84-P, IC2 ULN2803, P1 +V=VRx / +V<VRx, P10 OUTPUT_1X8_GND, P2 XANY_INPUT, P3 SERVO, P4 DIODE, P5 OUTPUT_1X8, P6 VExt, P7 OUTPUT_1X8_ALIM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

Commit message: Push of MS8 PCB folder for Pierrot :-)
Parts:
- R3: value 100 -> 1K
Other:
- note added: "- Load +"
- note added: "Servo"
- note added: "Signal + -"
Changed lines of the file:
@@
 Sheet 1 1
 Title "Décodeur MS8 X-Any"
-Date "2018-12-18"
+Date "2018-12-20"
 Rev "0.1"
 Comp "OpenAVRc"
@@
 P 2500 4550
 F 0 "R3" V 2580 4550 40  0000 C CNN
-F 1 "100" V 2507 4551 40  0000 C CNN
+F 1 "1K" V 2507 4551 40  0000 C CNN
 F 2 "R_1206" V 2430 4550 30  0001 C CNN
 F 3 "" H 2500 4550 30  0000 C CNN
@@
 Wire Wire Line
 	8700 3500 7850 3500
+Wire Notes Line
+	8950 2700 9050 2600
+Wire Notes Line
+	9050 2600 9600 2600
+Wire Notes Line
+	9600 2600 9700 2700
+Text Notes 9100 2550 0    60   ~ 0
+- Load +
+Wire Notes Line
+	8950 2500 9050 2400
+Wire Notes Line
+	9050 2400 10100 2400
+Wire Notes Line
+	10100 2400 10200 2500
+Text Notes 9050 2400 0    60   ~ 0
+Signal     +         -
+Text Notes 9450 2300 0    60   ~ 0
+Servo
 $EndSCHEMATC
