File: PCB/PCB Shield/Mega_2560 core mini_full_2.2_PM/OpenAVRc_Audio_Haptic.sch (KiCad schematic (older format))
At the start: 14 parts, among them P22 JQ6500_28P, P5 Vibreur, P8 Audio, Q2 MMBT2222ALT1

Commit message: Update PCB files V2.2
Move r5 after r6
Other:
- moved on the sheet: C20, C21, P22, R3, R4
