File: PCB/PCB Shield/Mega_2560 core mini_full_2.2_PM/OpenAVRc_HF_Telemetry.sch (KiCad schematic (older format))
At the start: 13 parts, among them P18 Ecolage, P19 Module_Tx, P20 TTL/RS232, P3 FTDI, P7 SPIX, U1 74LVC1G3157GV, U2 74LVC1G3157GV, U3 74LVC1G3157GV

Commit message: Update Shield v2.2
-Add pullup on Rx core
-Add 3D views TOP and BOTTOM
Parts:
- P20: footprint anthoperso:Con_RS232_TTL -> Mylib_v2.2:Con_RS232_TTL
- P7: footprint Pin_Headers:Pin_Header_Straight_2x05_Pitch2.54mm -> Mylib_v2.2:Pin_Header_Straight_2x05_Pitch2.54mm
- R18, R19, R7, R8: footprint Resistors_SMD:R_1206 -> Mylib_v2.2:R_1206
- U1, U2, U3: footprint v2.1:SOT-457 -> Mylib_v2.2:SOT-457
Changed lines of the file:
@@
 F 0 "R8" V 10030 4800 50  0000 C CNN
 F 1 "200" V 9950 4800 50  0000 C CNN
-F 2 "Resistors_SMD:R_1206" V 9880 4800 50  0001 C CNN
+F 2 "Mylib_v2.2:R_1206" V 9880 4800 50  0001 C CNN
 F 3 "" H 9950 4800 50  0000 C CNN
 	1    9950 4800
@@
 F 0 "P20" H 2100 5000 50  0000 C CNN
 F 1 "TTL/RS232" H 2100 4500 50  0000 C CNN
-F 2 "anthoperso:Con_RS232_TTL" H 1900 4550 50  0001 C CNN
+F 2 "Mylib_v2.2:Con_RS232_TTL" H 1900 4550 50  0001 C CNN
 F 3 "" H 1900 4550 50  0000 C CNN
 	1    1900 4550
@@
 F 0 "U1" H 8750 5050 60  0000 C CNN
 F 1 "74LVC1G3157GV" H 8750 4000 60  0000 C CNN
-F 2 "v2.1:SOT-457" H 8750 4500 60  0001 C CNN
+F 2 "Mylib_v2.2:SOT-457" H 8750 4500 60  0001 C CNN
 F 3 "" H 8750 4500 60  0000 C CNN
 	1    8750 4500
@@
 F 0 "P7" H 6950 1700 50  0000 C CNN
 F 1 "SPIX" V 6950 550 50  0000 C CNN
-F 2 "Pin_Headers:Pin_Header_Straight_2x05_Pitch2.54mm" H 6950 1150 50  0001 C CNN
+F 2 "Mylib_v2.2:Pin_Header_Straight_2x05_Pitch2.54mm" H 6950 1150 50  0001 C CNN
 F 3 "" H 6950 1150 50  0000 C CNN
 	1    6950 1150
@@
 F 0 "R18" V 3150 1850 50  0000 C CNN
 F 1 "200" V 3250 1850 50  0000 C CNN
-F 2 "Resistors_SMD:R_1206" V 3180 1850 50  0001 C CNN
+F 2 "Mylib_v2.2:R_1206" V 3180 1850 50  0001 C CNN
 F 3 "" H 3250 1850 50  0000 C CNN
 	1    3250 1850
@@
 F 0 "R19" V 5580 6000 50  0000 C CNN
 F 1 "220" V 5500 6000 50  0000 C CNN
-F 2 "Resistors_SMD:R_1206" V 5430 6000 50  0001 C CNN
+F 2 "Mylib_v2.2:R_1206" V 5430 6000 50  0001 C CNN
 F 3 "" H 5500 6000 50  0000 C CNN
 	1    5500 6000
@@
 F 0 "U2" H 4650 4950 60  0000 C CNN
 F 1 "74LVC1G3157GV" H 4650 3900 60  0000 C CNN
-F 2 "v2.1:SOT-457" H 4650 4400 60  0001 C CNN
+F 2 "Mylib_v2.2:SOT-457" H 4650 4400 60  0001 C CNN
 F 3 "" H 4650 4400 60  0000 C CNN
 	1    4650 4400
@@
 F 0 "U3" H 4650 6250 60  0000 C CNN
 F 1 "74LVC1G3157GV" H 4650 5200 60  0000 C CNN
-F 2 "v2.1:SOT-457" H 4650 5700 60  0001 C CNN
+F 2 "Mylib_v2.2:SOT-457" H 4650 5700 60  0001 C CNN
 F 3 "" H 4650 5700 60  0000 C CNN
 	1    4650 5700
@@
 F 0 "R7" V 5580 4700 50  0000 C CNN
 F 1 "220" V 5500 4700 50  0000 C CNN
-F 2 "Resistors_SMD:R_1206" V 5430 4700 50  0001 C CNN
+F 2 "Mylib_v2.2:R_1206" V 5430 4700 50  0001 C CNN
 F 3 "" H 5500 4700 50  0000 C CNN
 	1    5500 4700

Commit message: Update shield v2.2 3D views
Other:
- note added: "En cas d'absence du module\nTTL/RS232 connecter les pins:\n5 à 2 et 6 à 1."
Changed lines of the file:
@@
 	0    -1   -1   0
 $EndComp
+Text Notes 1400 5300 0    50   ~ 0
+En cas d'absence du module\nTTL/RS232 connecter les pins:\n5 à 2 et 6 à 1.
 $EndSCHEMATC
