File: PCB/PCB Shield/Mega_2560 core mini_full_2.2_PM/OpenAVRc_I2C.sch (KiCad schematic (older format))
At the start: 9 parts, among them P2 LCD_I2C, U7 FM24W256, U8 DS3231SN

Commit message: Update Shield v2.2
-Add pullup on Rx core
-Add 3D views TOP and BOTTOM
Parts:
- R15, R20: footprint Resistors_SMD:R_1206 -> Mylib_v2.2:R_1206
- U7: footprint v2.1:SOIC-8-FRAM_DI -> Mylib_v2.2:SOIC-8-FRAM_DI
- U8: footprint v2.1:SO-16-DS3231 -> Mylib_v2.2:SO-16-DS3231
Changed lines of the file:
@@
 F 0 "U7" H 8400 4400 60  0000 C CNN
 F 1 "FM24W256" H 8500 3700 60  0000 C CNN
-F 2 "v2.1:SOIC-8-FRAM_DI" H 8250 4050 60  0001 C CNN
+F 2 "Mylib_v2.2:SOIC-8-FRAM_DI" H 8250 4050 60  0001 C CNN
 F 3 "" H 8250 4050 60  0001 C CNN
 	1    8250 4050
@@
 F 0 "U8" H 5150 4650 60  0000 C CNN
 F 1 "DS3231SN" H 5150 3650 60  0000 C CNN
-F 2 "v2.1:SO-16-DS3231" H 5100 4100 60  0001 C CNN
+F 2 "Mylib_v2.2:SO-16-DS3231" H 5100 4100 60  0001 C CNN
 F 3 "" H 5100 4100 60  0001 C CNN
 	1    5150 4150
@@
 F 0 "R15" V 5780 3450 50  0000 C CNN
 F 1 "10K" V 5700 3450 50  0000 C CNN
-F 2 "Resistors_SMD:R_1206" V 5630 3450 50  0001 C CNN
+F 2 "Mylib_v2.2:R_1206" V 5630 3450 50  0001 C CNN
 F 3 "" H 5700 3450 50  0000 C CNN
 	1    5700 3450
@@
 F 0 "R20" V 5980 3450 50  0000 C CNN
 F 1 "10K" V 5900 3450 50  0000 C CNN
-F 2 "Resistors_SMD:R_1206" V 5830 3450 50  0001 C CNN
+F 2 "Mylib_v2.2:R_1206" V 5830 3450 50  0001 C CNN
 F 3 "" H 5900 3450 50  0000 C CNN
 	1    5900 3450
