File: PCB/PCB Shield/Mega_2560 core mini_full_2.2_PM/OpenAVRc_Power.sch (KiCad schematic (older format))
At the start: 24 parts, among them P17 BATT, P21 Sw_power, P26 LCD_Alim, P30 MiniDCDC3A, Q3 MMBT2222ALT1, Q4 SI2319DS, U4 PM5033, U5 LD1117S33TR

Commit message: Update Shield v2.2
-Add pullup on Rx core
-Add 3D views TOP and BOTTOM
Parts:
- P30: footprint v2.1:MiniDCDC3A -> Mylib_v2.2:MiniDCDC3A
- Q3: footprint v2.1:SOT-23_MMBT2222 -> Mylib_v2.2:SOT-23_MMBT2222
- Q4: footprint v2.1:SOT-23_MOS_P -> Mylib_v2.2:SOT-23_MOS_P
- R1, R16, R17, R2, R21, R22, R41, R42, R43: footprint Resistors_SMD:R_1206 -> Mylib_v2.2:R_1206
- U4: footprint v2.1:Pm5033_sil5 -> Mylib_v2.2:Pm5033_sil5
- U5: footprint TO_SOT_Packages_SMD:SOT-223 -> Mylib_v2.2:SOT-223
Changed lines of the file:
@@
 F 0 "R16" V 5730 4350 50  0000 C CNN
 F 1 "2.7K" V 5650 4350 50  0000 C CNN
-F 2 "Resistors_SMD:R_1206" V 5580 4350 50  0001 C CNN
+F 2 "Mylib_v2.2:R_1206" V 5580 4350 50  0001 C CNN
 F 3 "" H 5650 4350 50  0000 C CNN
 	1    5650 4350
@@
 F 0 "U5" H 9100 3800 50  0000 C CNN
 F 1 "LD1117S33TR" H 9300 4250 50  0000 C CNN
-F 2 "TO_SOT_Packages_SMD:SOT-223" H 9300 4150 50  0001 C CNN
+F 2 "Mylib_v2.2:SOT-223" H 9300 4150 50  0001 C CNN
 F 3 "" H 9300 4050 50  0000 C CNN
 	1    9300 4050
@@
 F 0 "R17" V 5730 3600 50  0000 C CNN
 F 1 "5.1K" V 5650 3600 50  0000 C CNN
-F 2 "Resistors_SMD:R_1206" V 5580 3600 50  0001 C CNN
+F 2 "Mylib_v2.2:R_1206" V 5580 3600 50  0001 C CNN
 F 3 "" H 5650 3600 50  0000 C CNN
 	1    5650 3600
@@
 F 0 "U4" H 7850 2850 60  0000 C CNN
 F 1 "PM5033" H 7650 3450 60  0000 C CNN
-F 2 "v2.1:Pm5033_sil5" H 7650 3150 60  0001 C CNN
+F 2 "Mylib_v2.2:Pm5033_sil5" H 7650 3150 60  0001 C CNN
 F 3 "" H 7650 3150 60  0000 C CNN
 	1    7650 3150
@@
 F 0 "R43" V 7080 3650 50  0000 C CNN
 F 1 "10K" V 7000 3650 50  0000 C CNN
-F 2 "Resistors_SMD:R_1206" V 6930 3650 50  0001 C CNN
+F 2 "Mylib_v2.2:R_1206" V 6930 3650 50  0001 C CNN
 F 3 "" H 7000 3650 50  0000 C CNN
 	1    7000 3650
@@
 F 0 "R41" V 6780 3300 50  0000 C CNN
 F 1 "33K" V 6700 3300 50  0000 C CNN
-F 2 "Resistors_SMD:R_1206" V 6630 3300 50  0001 C CNN
+F 2 "Mylib_v2.2:R_1206" V 6630 3300 50  0001 C CNN
 F 3 "" H 6700 3300 50  0000 C CNN
 	1    6700 3300
@@
 F 0 "Q4" V 4850 3300 60  0000 R CNN
 F 1 "SI2319DS" V 5250 3300 60  0000 R CNN
-F 2 "v2.1:SOT-23_MOS_P" H 5000 3100 60  0001 C CNN
+F 2 "Mylib_v2.2:SOT-23_MOS_P" H 5000 3100 60  0001 C CNN
 F 3 "" H 5000 3100 60  0000 C CNN
 	1    5000 3100
@@
 F 0 "Q3" H 4900 3950 50  0000 R CNN
 F 1 "MMBT2222ALT1" V 5100 4400 50  0000 R CNN
-F 2 "v2.1:SOT-23_MMBT2222" H 4900 4100 60  0001 C CNN
+F 2 "Mylib_v2.2:SOT-23_MMBT2222" H 4900 4100 60  0001 C CNN
 F 3 "" H 4900 4100 60  0000 C CNN
 	1    4900 4100
@@
 F 0 "R42" V 4680 3350 50  0000 C CNN
 F 1 "100K" V 4600 3350 50  0000 C CNN
-F 2 "Resistors_SMD:R_1206" V 4530 3350 50  0001 C CNN
+F 2 "Mylib_v2.2:R_1206" V 4530 3350 50  0001 C CNN
 F 3 "" H 4600 3350 50  0000 C CNN
 	1    4600 3350
@@
 F 0 "R1" V 5080 3650 50  0000 C CNN
 F 1 "5,1K" V 5000 3650 50  0000 C CNN
-F 2 "Resistors_SMD:R_1206" V 4930 3650 50  0001 C CNN
+F 2 "Mylib_v2.2:R_1206" V 4930 3650 50  0001 C CNN
 F 3 "" H 5000 3650 50  0000 C CNN
 	1    5000 3650
@@
 F 0 "R2" V 4030 4100 50  0000 C CNN
 F 1 "5,1K" V 3950 4100 50  0000 C CNN
-F 2 "Resistors_SMD:R_1206" V 3880 4100 50  0001 C CNN
+F 2 "Mylib_v2.2:R_1206" V 3880 4100 50  0001 C CNN
 F 3 "" H 3950 4100 50  0000 C CNN
 	1    3950 4100
@@
 F 0 "R22" V 4480 3750 50  0000 C CNN
 F 1 "8,2K" V 4400 3750 50  0000 C CNN
-F 2 "Resistors_SMD:R_1206" V 4330 3750 50  0001 C CNN
+F 2 "Mylib_v2.2:R_1206" V 4330 3750 50  0001 C CNN
 F 3 "" H 4400 3750 50  0000 C CNN
 	1    4400 3750
@@
 F 0 "R21" V 4730 4350 50  0000 C CNN
 F 1 "10K" V 4650 4350 50  0000 C CNN
-F 2 "Resistors_SMD:R_1206" V 4580 4350 50  0001 C CNN
+F 2 "Mylib_v2.2:R_1206" V 4580 4350 50  0001 C CNN
 F 3 "" H 4650 4350 50  0000 C CNN
 	1    4650 4350
@@
 F 0 "P30" H 2150 4600 50  0000 C CNN
 F 1 "MiniDCDC3A" V 2250 4200 50  0000 C CNN
-F 2 "v2.1:MiniDCDC3A" H 2150 4200 50  0001 C CNN
+F 2 "Mylib_v2.2:MiniDCDC3A" H 2150 4200 50  0001 C CNN
 F 3 "~" H 2150 4200 50  0001 C CNN
 	1    2150 4200
