File: PCB/MultiSwitch_MosFet/MultiSwitch_MosFet.kicad_pcb (KiCad board)
At the start: 2 copper layers, 77.5 x 57.2 mm, 71 parts, among them J1 VExt1, J10 VRx/Ms8, J11 VExt_GND, J2 VExt2, J3 VExt3, J4 VExt4, J5 VExt5, J6 VExt6, J7 VExt7, J8 VExt8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

Commit message: Add Texts
Other:
- board text added: "0V"
- board text added: "VRx+"
