File: PCB/PCB openXsensor/openXsensor.kicad_pcb (KiCad board)
At the start: 2 copper layers, 32.4 x 33 mm, 42 parts, among them P1 Digital, P10 VFAS/COURANT, P11 GY-86, P12 NTC1, P13 NTC2, P14 ALIM, P15 SEQUENCEUR, P16 4S, P17 ADS1115, P18 MS4525DO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

Commit message: Update oXs PCB proto
Parts:
- removed R2: 20K, R_1206
- removed R6: 51K, R_1206
- P10, P18, P5: footprint Pin_Header_Straight_1x04_Pitch2.54mm -> Empreintes:Pin_Header_Straight_1x04_Pitch2.54mm
- P11, P16: footprint Pin_Header_Straight_1x05_Pitch2.54mm -> Empreintes:Pin_Header_Straight_1x05_Pitch2.54mm
- P12, P13, P7: footprint Pin_Header_Straight_1x02_Pitch2.54mm -> Empreintes:Pin_Header_Straight_1x02_Pitch2.54mm
- P14, P19, P6, P8, P9: footprint Pin_Header_Straight_1x03_Pitch2.54mm -> Empreintes:Pin_Header_Straight_1x03_Pitch2.54mm
- P15: footprint Pin_Header_Straight_1x04_Pitch2.54mm -> Empreintes:Pin_Header_Straight_1x05_Pitch2.54mm
- P17: footprint Pin_Header_Straight_1x10_Pitch2.54mm -> Empreintes:Pin_Header_Straight_1x10_Pitch2.54mm
- R1, R10, R11: footprint R_1206 -> Empreintes:R_1206
- R3, R5: value 20K -> 10K; footprint R_1206 -> Empreintes:R_1206
- R4: value 20K -> 12K; footprint R_1206 -> Empreintes:R_1206
- R7: value 51K -> 8,2K; footprint R_1206 -> Empreintes:R_1206
- R8: value 51K -> 22K; footprint R_1206 -> Empreintes:R_1206
- R9: value 51K -> 27K; footprint R_1206 -> Empreintes:R_1206
- moved R3 4.47 mm to (143.5, 96.1), turned to 270 degrees
- moved R4 4.47 mm to (146.1, 96.1), turned to 270 degrees
- moved R5 4.47 mm to (148.6, 96.1), turned to 270 degrees
- moved R7 4.42 mm to (143.5, 91.6), turned to 270 degrees
- moved R8 4.42 mm to (146.1, 91.6), turned to 270 degrees
- moved R9 4.42 mm to (148.6, 91.6), turned to 270 degrees
- moved P6 2.54 mm to (135.3, 95.2)
- moved P7 2.54 mm to (135.3, 87.6)
- moved P15 2.54 mm to (135.3, 102.9)
Connections:
- C14 pad 1: /ADS_VOLT4 -> Net-(C14-Pad1)
- C7 pad 1: /ADS_VOLT3 -> Net-(C7-Pad1)
- C8 pad 1: /ADS_VOLT1 -> /A6
- C9 pad 1: /ADS_VOLT2 -> /A7
- P10 pad 3: /ADS_VOLT1 -> /A6
- P10 pad 4: /ADS_VOLT2 -> /A7
- P16 pad 1: Net-(P16-Pad1) -> GND
- P16 pad 2: Net-(P16-Pad2) -> /A0
- P16 pad 5: (no net) -> Net-(P16-Pad5)
- P17 pad 10: /ADS_VOLT4 -> (no net)
- P17 pad 7: /ADS_VOLT1 -> (no net)
- P17 pad 8: /ADS_VOLT2 -> (no net)
- P17 pad 9: /ADS_VOLT3 -> (no net)
- P19 pad 3: /ADS_VOLT3 -> Net-(C7-Pad1)
- P8 pad 1: /ADS_VOLT4 -> Net-(C14-Pad1)
- R7 pad 1: Net-(P16-Pad2) -> Net-(P16-Pad3)
- R8 pad 1: Net-(P16-Pad3) -> Net-(P16-Pad4)
- R9 pad 1: Net-(P16-Pad4) -> Net-(P16-Pad5)
Routing:
- net /ADS_VOLT4: track 22.6 -> 0.00 mm
- net /A6: track 10.2 -> 26.6 mm
- net /A7: track 12.0 -> 26.2 mm
- net Net-(P16-Pad2): track 10.9 -> 0.00 mm
- net /ADS_VOLT1: track 10.7 -> 0.00 mm
- net /ADS_VOLT2: track 10.7 -> 0.00 mm
- net Net-(P16-Pad4): track 10.9 -> 4.04 mm
- net Net-(P16-Pad3): track 10.9 -> 4.04 mm
- net /ADS_VOLT3: track 6.77 -> 0.00 mm
- net Net-(C14-Pad1): track 0.00 -> 5.63 mm
- net Net-(C7-Pad1): track 0.00 -> 4.97 mm
- net /A0: track 25.6 -> 29.8 mm, vias 1 -> 0
- net Net-(P16-Pad5): track 0.00 -> 4.04 mm
- net Net-(P16-Pad1): track 2.54 -> 0.00 mm
- net Net-(P6-Pad2): track 15.0 -> 17.4 mm
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