File: PCB/PCB openXsensor/openXsensor.sch (KiCad schematic (older format))
At the start: 42 parts, among them P1 Digital, P10 VFAS/COURANT, P11 GY-86, P12 NTC1, P13 NTC2, P14 ALIM, P15 SEQUENCEUR, P16 4S, P17 ADS1115, P18 MS4525DO, P19 MPXV7002DP, P2 Analog, P3 ADC, P4 ADC, P5 GPS, P6 HUB/SPORT, P7 PPM, P8 FUEL, P9 RPM

Commit message: Update oXs PCB proto
Parts:
- removed P15: SEQUENCEUR, Empreintes:Pin_Header_Straight_1x04_Pitch2.54mm, symbol Connector_Generic:Conn_01x04
- removed R2: 20K, Empreintes:R_1206, symbol Device:R
- removed R6: 51K, Empreintes:R_1206, symbol Device:R
- added P15: SEQUENCEUR, Empreintes:Pin_Header_Straight_1x05_Pitch2.54mm, symbol Connector_Generic:Conn_01x05
- R3, R5: value 20K -> 10K
- R4: value 20K -> 12K
- R7: value 51K -> 8,2K
- R8: value 51K -> 22K
- R9: value 51K -> 27K
Connections:
- net labels removed: CURRENT, VFAS
- wire segments 161 -> 153
Other:
- moved on the sheet: R7, R8, R9
Changed lines of the file:
@@
 EESchema Schematic File Version 4
-LIBS:openXsensor-cache
-EELAYER 26 0
+EELAYER 30 0
 EELAYER END
 $Descr A4 11693 8268
@@
 F 3 "~" H 2550 3650 50  0001 C CNN
 	1    2550 3650
-	-1   0    0    -1
+	-1   0    0    1
 $EndComp
 $Comp
@@
 Wire Wire Line
 	7150 3300 7400 3300
-$Comp
-L Device:R R6
-U 1 1 5D92216D
-P 3050 3450
-F 0 "R6" V 3000 3250 50  0000 C CNN
-F 1 "51K" V 3050 3450 50  0000 C CNN
-F 2 "Empreintes:R_1206" V 2980 3450 50  0001 C CNN
-F 3 "~" H 3050 3450 50  0001 C CNN
-	1    3050 3450
-	0    -1   1    0
-$EndComp
-$Comp
-L Device:R R2
-U 1 1 5D922625
-P 3400 4000
-F 0 "R2" V 3350 3800 50  0000 C CNN
-F 1 "20K" V 3400 4000 50  0000 C CNN
-F 2 "Empreintes:R_1206" V 3330 4000 50  0001 C CNN
-F 3 "~" H 3400 4000 50  0001 C CNN
-	1    3400 4000
-	-1   0    0    -1
-$EndComp
 Wire Wire Line
 	3700 4150 3700 4250
@@
 	3700 4250 3600 4250
 Wire Wire Line
-	3400 4250 3400 4150
-Wire Wire Line
 	3500 4150 3500 4250
-Connection ~ 3500 4250
-Wire Wire Line
-	3500 4250 3400 4250
 Wire Wire Line
 	3600 4150 3600 4250
@@
 	-1   0    0    -1
 $EndComp
-Wire Wire Line
-	3700 3750 3700 3850
-Wire Wire Line
-	3600 3650 3600 3850
-Wire Wire Line
-	3500 3550 3500 3850
-Wire Wire Line
-	3400 3450 3400 3850
 Text Label 4650 3450 0    50   ~ 0
-A0
+A3
 Text Label 4650 3550 0    50   ~ 0
-A1
-Text Label 4650 3650 0    50   ~ 0
 A2
+Text Label 4650 3650 0    50   ~ 0
+A1
 Text Label 4650 3750 0    50   ~ 0
-A3
+A0
 $Comp
 L Device:R R7
 U 1 1 5D95CD07
-P 3050 3550
-F 0 "R7" V 3000 3350 50  0000 C CNN
-F 1 "51K" V 3050 3550 50  0000 C CNN
-F 2 "Empreintes:R_1206" V 2980 3550 50  0001 C CNN
-F 3 "~" H 3050 3550 50  0001 C CNN
-	1    3050 3550
+P 3050 3650
+F 0 "R7" V 3000 3450 50  0000 C CNN
+F 1 "8,2K" V 3050 3650 50  0000 C CNN
+F 2 "Empreintes:R_1206" V 2980 3650 50  0001 C CNN
+F 3 "~" H 3050 3650 50  0001 C CNN
+	1    3050 3650
 	0    -1   1    0
 $EndComp
@@
 L Device:R R8
 U 1 1 5D95CD3F
-P 3050 3650
-F 0 "R8" V 3000 3450 50  0000 C CNN
-F 1 "51K" V 3050 3650 50  0000 C CNN
-F 2 "Empreintes:R_1206" V 2980 3650 50  0001 C CNN
-F 3 "~" H 3050 3650 50  0001 C CNN
-	1    3050 3650
+P 3050 3550
+F 0 "R8" V 3000 3350 50  0000 C CNN
+F 1 "22K" V 3050 3550 50  0000 C CNN
+F 2 "Empreintes:R_1206" V 2980 3550 50  0001 C CNN
+F 3 "~" H 3050 3550 50  0001 C CNN
+	1    3050 3550
 	0    -1   1    0
 $EndComp
@@
 L Device:R R9
 U 1 1 5D95CD7D
-P 3050 3750
-F 0 "R9" V 3000 3550 50  0000 C CNN
-F 1 "51K" V 3050 3750 50  0000 C CNN
-F 2 "Empreintes:R_1206" V 2980 3750 50  0001 C CNN
-F 3 "~" H 3050 3750 50  0001 C CNN
-	1    3050 3750
+P 3050 3450
+F 0 "R9" V 3000 3250 50  0000 C CNN
+F 1 "27K" V 3050 3450 50  0000 C CNN
+F 2 "Empreintes:R_1206" V 2980 3450 50  0001 C CNN
+F 3 "~" H 3050 3450 50  0001 C CNN
+	1    3050 3450
 	0    -1   1    0
 $EndComp
@@
 P 3500 4000
 F 0 "R3" V 3450 3800 50  0000 C CNN
-F 1 "20K" V 3500 4000 50  0000 C CNN
+F 1 "10K" V 3500 4000 50  0000 C CNN
 F 2 "Empreintes:R_1206" V 3430 4000 50  0001 C CNN
 F 3 "~" H 3500 4000 50  0001 C CNN
@@
 P 3600 4000
 F 0 "R4" V 3550 3800 50  0000 C CNN
-F 1 "20K" V 3600 4000 50  0000 C CNN
+F 1 "12K" V 3600 4000 50  0000 C CNN
 F 2 "Empreintes:R_1206" V 3530 4000 50  0001 C CNN
 F 3 "~" H 3600 4000 50  0001 C CNN
@@
 P 3700 4000
 F 0 "R5" V 3650 3800 50  0000 C CNN
-F 1 "20K" V 3700 4000 50  0000 C CNN
+F 1 "10K" V 3700 4000 50  0000 C CNN
 F 2 "Empreintes:R_1206" V 3630 4000 50  0001 C CNN
 F 3 "~" H 3700 4000 50  0001 C CNN
@@
 RAW
 Wire Wire Line
-	2900 3450 2750 3450
-Wire Wire Line
-	3200 3450 3400 3450
-Connection ~ 3400 3450
-Wire Wire Line
-	3200 3550 3500 3550
-Connection ~ 3500 3550
-Wire Wire Line
-	3200 3650 3600 3650
-Connection ~ 3600 3650
-Wire Wire Line
-	3200 3750 3700 3750
-Connection ~ 3700 3750
-Wire Wire Line
 	2900 3550 2750 3550
 Wire Wire Line
 	2900 3650 2750 3650
-Wire Wire Line
-	2900 3750 2750 3750
-Wire Wire Line
-	3400 3450 3850 3450
-Wire Wire Line
-	3500 3550 4100 3550
-Wire Wire Line
-	3600 3650 4350 3650
-Wire Wire Line
-	3700 3750 4600 3750
 $Comp
 L Device:R R10
@@
 Text Label 4100 7250 0    50   ~ 0
 A7
-Text Label 2800 5550 0    50   ~ 0
-VFAS
-Text Label 2800 5650 0    50   ~ 0
-CURRENT
 $Comp
 L Device:C C1
@@
 $EndComp
 Wire Wire Line
-	3850 3800 3850 3450
-Connection ~ 3850 3450
-Wire Wire Line
-	3850 3450 4650 3450
-Wire Wire Line
 	3850 4100 3850 4250
 $Comp
@@
 	4600 4100 4600 4250
 Wire Wire Line
-	4100 3800 4100 3550
-Connection ~ 4100 3550
-Wire Wire Line
-	4100 3550 4650 3550
-Wire Wire Line
-	4350 3800 4350 3650
-Connection ~ 4350 3650
-Wire Wire Line
-	4350 3650 4650 3650
-Wire Wire Line
-	4600 3800 4600 3750
-Connection ~ 4600 3750
-Wire Wire Line
-	4600 3750 4650 3750
-Wire Wire Line
 	3850 4250 4100 4250
 Connection ~ 4100 4250
@@
 	3800 6650 3650 6650
 Wire Wire Line
-	2750 5650 3400 5650
-Wire Wire Line
 	3350 2800 3350 2700
 Wire Wire Line
@@
 	3250 7250 4100 7250
 Wire Wire Line
-	3300 5550 3300 5200
-Connection ~ 3300 5200
-Wire Wire Line
-	3300 5200 3300 4750
-Wire Wire Line
 	3300 5200 3700 5200
 $Comp
@@
 Wire Wire Line
 	4000 5950 4250 5950
-Wire Wire Line
-	3400 4850 3400 5650
-Wire Wire Line
-	3700 5650 3400 5650
-Connection ~ 3400 5650
-Wire Wire Line
-	2750 5950 3600 5950
-Wire Wire Line
-	3500 4950 3500 6450
-Wire Wire Line
-	3600 5050 3600 5950
-Connection ~ 3600 5950
-Wire Wire Line
-	3600 5950 3700 5950
 $Bitmap
 Pos 1350 6500
@@
 Data
 89 50 4E 47 0D 0A 1A 0A 00 00 00 0D 49 48 44 52 00 00 00 BE 00 00 00 76 08 02 00 00 00 F9 AD BE
-13 00 00 00 03 73 42 49 54 08 08 08 DB E1 4F E0 00 00 00 09 70 48 59 73 00 00 0E C3 00 00 0E C3
-01 C7 6F A8 64 00 00 20 00 49 44 41 54 78 9C ED 5D D9 6F 64 77 56 FE 6D 77 BF B7 6E 6D B6 CB 76
+13 00 00 00 03 73 42 49 54 08 08 08 DB E1 4F E0 00 00 00 09 70 48 59 73 00 00 0E 74 00 00 0E 74
+01 6B 24 B3 D6 00 00 20 00 49 44 41 54 78 9C ED 5D D9 6F 64 77 56 FE 6D 77 BF B7 6E 6D B6 CB 76
 DB EE 2D 49 67 61 94 21 62 18 A2 81 CC A0 61 20 C0 0C 42 42 2C 42 02 1E 10 91 90 18 09 89 47 D0
 84 FF 04 5E 90 90 10 0F 20 22 A4 84 59 49 20 E9 EC DD 9D 76 F7 B8 BB 6D 97 CB 65 BB F6 E5 EE 1B
@@
 Text Notes 3100 1500 0    50   ~ 0
 STRAP
-$Comp
-L Connector_Generic:Conn_01x04 P15
-U 1 1 5DB43FB7
-P 5950 4700
-F 0 "P15" H 5950 4900 50  0000 C CNN
-F 1 "SEQUENCEUR" H 6300 4650 50  0000 C CNN
-F 2 "Empreintes:Pin_Header_Straight_1x04_Pitch2.54mm" H 5950 4700 50  0001 C CNN
-F 3 "~" H 5950 4700 50  0001 C CNN
-	1    5950 4700
-	-1   0    0    -1
-$EndComp
 Wire Wire Line
 	6150 4600 6500 4600
@@
 Text Label 6500 4600 0    60   ~ 0
 SEQ4
+$Comp
+L Connector_Generic:Conn_01x05 P15
+U 1 1 5DB62DCC
+P 5950 4800
+F 0 "P15" H 5850 5100 50  0000 L CNN
+F 1 "SEQUENCEUR" H 6050 4800 50  0000 L CNN
+F 2 "Empreintes:Pin_Header_Straight_1x05_Pitch2.54mm" H 5950 4800 50  0001 C CNN
+F 3 "~" H 5950 4800 50  0001 C CNN
+	1    5950 4800
+	-1   0    0    -1
+$EndComp
+$Comp
+L power:GND #PWR0130
+U 1 1 5DB63140
+P 6300 5000
+F 0 "#PWR0130" H 6300 4750 50  0001 C CNN
+F 1 "GND" V 6300 4800 50  0000 C CNN
+F 2 "" H 6300 5000 50  0000 C CNN
+F 3 "" H 6300 5000 50  0000 C CNN
+	1    6300 5000
+	0    -1   -1   0
+$EndComp
+Wire Wire Line
+	6150 5000 6300 5000
+Wire Wire Line
+	2750 3850 2800 3850
+Wire Wire Line
+	2800 3850 2800 3900
+$Comp
+L power:GND #PWR0133
+U 1 1 5EF24BBF
+P 2800 3900
+F 0 "#PWR0133" H 2800 3650 50  0001 C CNN
+F 1 "GND" H 2800 3750 50  0000 C CNN
+F 2 "" H 2800 3900 50  0000 C CNN
+F 3 "" H 2800 3900 50  0000 C CNN
+	1    2800 3900
+	1    0    0    -1
+$EndComp
+Wire Wire Line
+	4650 3450 4600 3450
+Wire Wire Line
+	2900 3450 2750 3450
+Wire Wire Line
+	3200 3550 3600 3550
+Wire Wire Line
+	3200 3650 3500 3650
+Wire Wire Line
+	3700 3850 3700 3450
+Connection ~ 3700 3450
+Wire Wire Line
+	3700 3450 3200 3450
+Wire Wire Line
+	3600 3850 3600 3550
+Connection ~ 3600 3550
+Wire Wire Line
+	3500 3850 3500 3650
+Connection ~ 3500 3650
+Wire Wire Line
+	3600 3550 4350 3550
+Wire Wire Line
+	3500 3650 4100 3650
+Wire Wire Line
+	4600 3800 4600 3450
+Connection ~ 4600 3450
+Wire Wire Line
+	4600 3450 3700 3450
+Wire Wire Line
+	4350 3800 4350 3550
+Connection ~ 4350 3550
+Wire Wire Line
+	4350 3550 4650 3550
+Wire Wire Line
+	4100 3800 4100 3650
+Connection ~ 4100 3650
+Wire Wire Line
+	4100 3650 4650 3650
+Wire Wire Line
+	3850 3800 3850 3750
+Connection ~ 3850 3750
+Wire Wire Line
+	3850 3750 4650 3750
+Wire Wire Line
+	2750 3750 3850 3750
+Wire Wire Line
+	2750 5650 3700 5650
+Text Label 3150 5550 0    50   ~ 0
+A6
+Text Label 3150 5650 0    50   ~ 0
+A7
+Wire Wire Line
+	3300 5200 3300 5550
+Wire Wire Line
+	2750 5950 3700 5950
 $EndSCHEMATC

Commit message: Update oXs & add Gerber files
Parts:
- P11: value GY-86 -> VARIO
Other:
- note added: "(0x77)"
- note added: "ACCUS"
- note added: "GY-86\nGY-63\nBMPXXX"
Changed lines of the file:
@@
 Sheet 1 1
 Title ""
-Date "2019-10-19"
+Date "2020-06-19"
 Rev ""
 Comp ""
@@
 P 2550 2900
 F 0 "P11" H 2450 3200 50  0000 L CNN
-F 1 "GY-86" H 2650 2900 50  0000 L CNN
+F 1 "VARIO" H 2450 2600 50  0000 L CNN
 F 2 "Empreintes:Pin_Header_Straight_1x05_Pitch2.54mm" H 2550 2900 50  0001 C CNN
 F 3 "~" H 2550 2900 50  0001 C CNN
@@
 U 1 1 5D771791
 P 2550 3650
-F 0 "P16" H 2450 3950 50  0000 L CNN
-F 1 "4S" H 2650 3650 50  0000 L CNN
+F 0 "P16" H 2450 3350 50  0000 L CNN
+F 1 "4S" H 2700 3500 50  0000 L CNN
 F 2 "Empreintes:Pin_Header_Straight_1x05_Pitch2.54mm" H 2550 3650 50  0001 C CNN
 F 3 "~" H 2550 3650 50  0001 C CNN
@@
 Wire Wire Line
 	2750 5950 3700 5950
+Text Notes 2150 2950 0    50   ~ 0
+GY-86\nGY-63\nBMPXXX
+Text Notes 2200 3700 0    50   ~ 0
+ACCUS
+Text Notes 2150 3050 0    50   ~ 0
+(0x77)
 $EndSCHEMATC
