File: PCB/MultiSwitch_Sw16-ProMicro/MultiSwitch_Sw16_ProMicro.kicad_pcb (KiCad board)
At the start: 2 copper layers, 92.1 x 59.7 mm, 69 parts, among them J1 RC-, J10 X09T-X16T, J11 X09+-X16+, J12 X09--X16-, J13 DIODE2, J14 POW2_SEL, J15 VCPU_SEL, J16 Power, J17 +ExtV1_Out, J18 +ExtV1_In, J19 GND, J2 RC+, J20 Power1, J21 Power2, J22 +Ext2_In, J23 GND, J25 +Ext2_Out, J3 RCS, J4 X01--X08-, J5 X01+-X08+, J6 X01T-X08T, J7 POW1_SEL, J8 SERVO PROP, J9 DIODE1, P1 Digital, P2 Analog, Q1 BC337, U1 ULN2803A, U2 ULN2803A, U3 LM2596_DC-DC, U4 LM2596_DC-DC

Commit message: Update PCB Ms8 & Ms16 Pro Micro
Update Past Mask
Other:
- board text added: "A"
- board text added: "K"
Changed lines of the file:
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@@
   (general
     (thickness 1.6)
-    (drawings 89)
+    (drawings 103)
     (tracks 281)
     (zones 0)
@@
   (layers
     (0 F.Cu signal hide)
-    (31 B.Cu signal)
+    (31 B.Cu signal hide)
     (32 B.Adhes user hide)
     (33 F.Adhes user hide)
     (34 B.Paste user hide)
     (35 F.Paste user hide)
-    (36 B.SilkS user)
+    (36 B.SilkS user hide)
     (37 F.SilkS user hide)
     (38 B.Mask user hide)
-    (39 F.Mask user hide)
+    (39 F.Mask user)
     (40 Dwgs.User user hide)
     (41 Cmts.User user hide)
     (42 Eco1.User user hide)
     (43 Eco2.User user hide)
-    (44 Edge.Cuts user)
+    (44 Edge.Cuts user hide)
     (45 Margin user hide)
     (46 B.CrtYd user hide)
     (47 F.CrtYd user hide)
-    (48 B.Fab user)
-    (49 F.Fab user)
+    (48 B.Fab user hide)
+    (49 F.Fab user hide)
   )
   (setup
@@
     (visible_elements 7FFFFFFF)
     (pcbplotparams
-      (layerselection 0x10000_7ffffffe)
+      (layerselection 0x000c0_7ffffffe)
       (usegerberextensions false)
       (usegerberattributes false)
       (usegerberadvancedattributes false)
       (creategerberjobfile false)
-      (excludeedgelayer false)
+      (excludeedgelayer true)
       (linewidth 0.100000)
       (plotframeref false)
@@
       (padsonsilk true)
       (subtractmaskfromsilk false)
-      (outputformat 4)
-      (mirror true)
+      (outputformat 1)
+      (mirror false)
       (drillshape 0)
       (scaleselection 1)
@@
     )
   )
+  (gr_line (start 187.96 130.81) (end 187.96 71.12) (layer B.Mask) (width 0.5))
+  (gr_line (start 166.37 130.81) (end 166.37 71.12) (layer B.Mask) (width 0.5))
+  (gr_line (start 111.76 71.12) (end 111.76 130.81) (layer B.Mask) (width 0.5))
+  (gr_line (start 203.835 71.12) (end 111.76 71.12) (layer B.Mask) (width 0.5))
+  (gr_line (start 203.835 130.81) (end 203.835 71.12) (layer B.Mask) (width 0.5))
+  (gr_line (start 111.76 130.81) (end 203.835 130.81) (layer B.Mask) (width 0.5))
+  (gr_line (start 187.96 130.81) (end 187.96 71.12) (layer F.Mask) (width 0.5))
+  (gr_line (start 166.37 130.81) (end 166.37 71.12) (layer F.Mask) (width 0.5))
+  (gr_line (start 111.76 71.12) (end 111.76 130.81) (layer F.Mask) (width 0.5))
+  (gr_line (start 203.835 71.12) (end 111.76 71.12) (layer F.Mask) (width 0.5))
+  (gr_line (start 203.835 130.81) (end 203.835 71.12) (layer F.Mask) (width 0.5))
+  (gr_line (start 111.76 130.81) (end 203.835 130.81) (layer F.Mask) (width 0.5))
+  (gr_text A (at 115.57 117.475 90) (layer F.SilkS)
+    (effects (font (size 1.5 1.5) (thickness 0.3)))
+  )
+  (gr_text K (at 117.856 123.444 90) (layer F.SilkS)
+    (effects (font (size 1.5 1.5) (thickness 0.3)))
+  )
   (dimension 3.81 (width 0.15) (layer F.Fab)
